File: Circuit/FNE/FNE.sch (KiCad schematic (older format))
At the start: 19 parts, among them J1 Conn_01x14_Female, J2 Conn_01x14_Female, J3 S8B-XH-A-1_LF__SN_, J4 S8B-XH-A-1_LF__SN_, U1 MAX485E

Commit message: eeprom
Parts:
- removed R12, R13, R14, R15, R16, R17, R18, R19, R20: 1Meg, symbol Device:R
Connections:
- wire segments 126 -> 114
Changed lines of the file:
@@
 Wire Wire Line
 	9850 4800 9850 4900
-Connection ~ 9850 4900
 Wire Wire Line
 	7750 4750 7850 4750
@@
 Wire Wire Line
 	7850 4550 7750 4550
-Wire Wire Line
-	9300 4600 9300 4250
 $Comp
 L power:+5V #PWR04
@@
 $EndComp
 Wire Wire Line
-	7850 4600 9300 4600
-Wire Wire Line
-	7850 4800 9750 4800
-Wire Wire Line
-	7850 4900 9850 4900
-Wire Wire Line
-	7850 5000 9850 5000
+	7800 4600 7850 4600
+Wire Wire Line
+	7800 4800 7850 4800
+Wire Wire Line
+	7800 4900 7850 4900
+Wire Wire Line
+	7800 5000 7850 5000
 Wire Wire Line
 	8300 2800 8600 2800
@@
 	8300 3350 7550 3350
 Wire Wire Line
-	8850 3800 8900 3800
-Wire Wire Line
-	7850 3800 8550 3800
-$Comp
-L Device:R R12
-U 1 1 5F71280A
-P 8700 3800
-F 0 "R12" V 8650 4000 50  0000 C CNN
-F 1 "1Meg" V 8650 4200 50  0000 C CNN
-F 2 "" V 8630 3800 50  0001 C CNN
-F 3 "~" H 8700 3800 50  0001 C CNN
-	1    8700 3800
-	0    -1   1    0
-$EndComp
-Wire Wire Line
-	8850 3900 8900 3900
-Wire Wire Line
-	7850 3900 8550 3900
-$Comp
-L Device:R R13
-U 1 1 5F7161A4
-P 8700 3900
-F 0 "R13" V 8650 4100 50  0000 C CNN
-F 1 "1Meg" V 8650 4300 50  0000 C CNN
-F 2 "" V 8630 3900 50  0001 C CNN
-F 3 "~" H 8700 3900 50  0001 C CNN
-	1    8700 3900
-	0    -1   1    0
-$EndComp
-Wire Wire Line
-	8850 4000 8900 4000
-Wire Wire Line
-	7850 4000 8550 4000
-$Comp
-L Device:R R14
-U 1 1 5F719CFC
-P 8700 4000
-F 0 "R14" V 8650 4200 50  0000 C CNN
-F 1 "1Meg" V 8650 4400 50  0000 C CNN
-F 2 "" V 8630 4000 50  0001 C CNN
-F 3 "~" H 8700 4000 50  0001 C CNN
-	1    8700 4000
-	0    -1   1    0
-$EndComp
-Wire Wire Line
-	8850 4100 8900 4100
-Wire Wire Line
-	7850 4100 8550 4100
-$Comp
-L Device:R R15
-U 1 1 5F71DA21
-P 8700 4100
-F 0 "R15" V 8650 4300 50  0000 C CNN
-F 1 "1Meg" V 8650 4500 50  0000 C CNN
-F 2 "" V 8630 4100 50  0001 C CNN
-F 3 "~" H 8700 4100 50  0001 C CNN
-	1    8700 4100
-	0    -1   1    0
-$EndComp
-Wire Wire Line
-	8850 4200 8900 4200
-Wire Wire Line
-	7850 4200 8550 4200
-$Comp
-L Device:R R16
-U 1 1 5F721992
-P 8700 4200
-F 0 "R16" V 8650 4400 50  0000 C CNN
-F 1 "1Meg" V 8650 4600 50  0000 C CNN
-F 2 "" V 8630 4200 50  0001 C CNN
-F 3 "~" H 8700 4200 50  0001 C CNN
-	1    8700 4200
-	0    -1   1    0
-$EndComp
-Wire Wire Line
-	8850 4300 8900 4300
-Wire Wire Line
-	7850 4300 8550 4300
-$Comp
-L Device:R R17
-U 1 1 5F725B5E
-P 8700 4300
-F 0 "R17" V 8650 4500 50  0000 C CNN
-F 1 "1Meg" V 8650 4700 50  0000 C CNN
-F 2 "" V 8630 4300 50  0001 C CNN
-F 3 "~" H 8700 4300 50  0001 C CNN
-	1    8700 4300
-	0    -1   1    0
-$EndComp
+	7800 3800 7850 3800
+Wire Wire Line
+	7800 3900 7850 3900
+Wire Wire Line
+	7800 4000 7850 4000
+Wire Wire Line
+	7800 4100 7850 4100
+Wire Wire Line
+	7800 4200 7850 4200
+Wire Wire Line
+	7800 4300 7850 4300
 Wire Wire Line
 	7950 4350 7850 4350
 Wire Wire Line
-	8850 4400 8900 4400
-Wire Wire Line
-	7850 4400 8550 4400
-$Comp
-L Device:R R18
-U 1 1 5F73365F
-P 8700 4400
-F 0 "R18" V 8650 4600 50  0000 C CNN
-F 1 "1Meg" V 8650 4800 50  0000 C CNN
-F 2 "" V 8630 4400 50  0001 C CNN
-F 3 "~" H 8700 4400 50  0001 C CNN
-	1    8700 4400
-	0    -1   1    0
-$EndComp
-Wire Wire Line
-	8850 4500 8900 4500
-Wire Wire Line
-	7850 4500 8550 4500
-$Comp
-L Device:R R19
-U 1 1 5F737C8B
-P 8700 4500
-F 0 "R19" V 8650 4700 50  0000 C CNN
-F 1 "1Meg" V 8650 4900 50  0000 C CNN
-F 2 "" V 8630 4500 50  0001 C CNN
-F 3 "~" H 8700 4500 50  0001 C CNN
-	1    8700 4500
-	0    -1   1    0
-$EndComp
+	7800 4400 7850 4400
+Wire Wire Line
+	7800 4500 7850 4500
 Wire Wire Line
 	8850 5100 8900 5100
 Wire Wire Line
-	7850 5100 8550 5100
-$Comp
-L Device:R R20
-U 1 1 5F73C5D9
-P 8700 5100
-F 0 "R20" V 8650 5300 50  0000 C CNN
-F 1 "1Meg" V 8650 5500 50  0000 C CNN
-F 2 "" V 8630 5100 50  0001 C CNN
-F 3 "~" H 8700 5100 50  0001 C CNN
-	1    8700 5100
-	0    -1   1    0
-$EndComp
+	7800 5100 7850 5100
 $Comp
 L power:GND #PWR03
@@
 	1    0    0    -1
 $EndComp
-Wire Wire Line
-	8900 3800 8900 3900
-Connection ~ 8900 3900
-Wire Wire Line
-	8900 3900 8900 4000
-Connection ~ 8900 4000
-Wire Wire Line
-	8900 4000 8900 4100
-Connection ~ 8900 4100
-Wire Wire Line
-	8900 4100 8900 4200
-Connection ~ 8900 4200
-Wire Wire Line
-	8900 4200 8900 4300
-Connection ~ 8900 4300
-Wire Wire Line
-	8900 4300 8900 4400
-Connection ~ 8900 4400
-Wire Wire Line
-	8900 4400 8900 4500
-Connection ~ 8900 4500
-Wire Wire Line
-	8900 4500 8900 4700
 Connection ~ 8900 5100
 Wire Wire Line
@@
 	7850 5050 7750 5050
 Wire Wire Line
-	7850 4700 8900 4700
-Connection ~ 8900 4700
+	7800 4700 7850 4700
 Wire Wire Line
 	8900 4700 8900 5100
@@
 	0    1    1    0
 $EndComp
-Wire Wire Line
-	9300 4600 9300 4700
-Connection ~ 9300 4600
 Wire Wire Line
 	9000 4700 8900 4700
@@
 	-1   0    0    -1
 $EndComp
+Connection ~ 7850 4600
+Wire Wire Line
+	7850 4600 9250 4600
+Connection ~ 7850 4700
+Wire Wire Line
+	7850 4700 8850 4700
+Connection ~ 7850 4800
+Wire Wire Line
+	7850 4800 9700 4800
+Connection ~ 7850 4900
+Wire Wire Line
+	7850 4900 9800 4900
+Connection ~ 7850 5000
+Wire Wire Line
+	7850 5000 9800 5000
+Wire Wire Line
+	9300 4250 9300 4700
 $EndSCHEMATC
