File: Circuit/terminal4N/terminal4N.sch (KiCad schematic (older format))
At the start: 10 parts, among them J1 Conn_01x05_Male, J2 Conn_02x08_Odd_Even, J3 Conn_01x02_Male, U1 4051

Commit message: ECM対策
Parts:
- added C3: 0.1u, Capacitor_THT:C_Disc_D3.0mm_W1.6mm_P2.50mm, symbol Device:C
- added R10, R11, R12, R13, R14, R15, R16, R9: 220, Resistor_THT:R_Axial_DIN0204_L3.6mm_D1.6mm_P7.62mm_Horizontal, symbol Device:R
- added U2: 74HC00, symbol 74xx:74HC00
Connections:
- net GND: now also C3.1, U2.10, U2.12, U2.13, U2.4, U2.5, U2.7 (GND), U2.9; no longer U1.6 (Inh)
- net VDD: now also C3.2, U2.14 (VCC)
- net at J2.1 (Pin_1), R8.1: now also R16.2; no longer U1.4 (X7)
- net at J2.10 (Pin_10): now also J2.11 (Pin_11), J2.12 (Pin_12), J2.13 (Pin_13), J2.14 (Pin_14), J2.15 (Pin_15), J2.16 (Pin_16), J2.2 (Pin_2), J2.4 (Pin_4), J2.6 (Pin_6), J2.8 (Pin_8), J2.9 (Pin_9), J3.2 (Pin_2), R5.2, R6.2, R7.2, R8.2, R10.2, R11.2, R12.2, R9.2
- net at J2.3 (Pin_3), R7.1: now also R15.2; no longer U1.2 (X6)
- net at J2.5 (Pin_5), R6.1: now also R14.2; no longer U1.5 (X5)
- net at J2.7 (Pin_7), R5.1: now also R13.2; no longer U1.1 (X4)
- net at U1.12 (X3): now also R12.1
- net at U1.13 (X0): now also R9.1
- net at U1.14 (X1): now also R10.1
- net at U1.15 (X2): now also R11.1
- net at J1.5 (Pin_5), U1.9 (C): now also U2.1, U2.2
- new net: U1.6 (Inh), U2.3
- new net: R13.1, U1.1 (X4)
- new net: R14.1, U1.5 (X5)
- new net: R15.1, U1.2 (X6)
- new net: R16.1, U1.4 (X7)
- no-connect marks 12 -> 3
Other:
- moved on the sheet: C2, J3, U1
