File: Circuit/terminal4S/terminal4S.sch (KiCad schematic (older format))
At the start: 10 parts, among them J1 Conn_01x05_Male, J2 Conn_02x08_Odd_Even, J3 Conn_01x02_Male, U1 4051

Commit message: ECM対策
Parts:
- added R10, R11, R12, R13, R14, R15, R16, R9: 220, Resistor_THT:R_Axial_DIN0204_L3.6mm_D1.6mm_P7.62mm_Horizontal, symbol Device:R
Connections:
- net GND: no longer U1.6 (Inh)
- net at J2.1 (Pin_1): now also J2.10 (Pin_10), J2.12 (Pin_12), J2.14 (Pin_14), J2.16 (Pin_16), J2.2 (Pin_2), J2.3 (Pin_3), J2.4 (Pin_4), J2.5 (Pin_5), J2.6 (Pin_6), J2.7 (Pin_7), J2.8 (Pin_8), J3.2 (Pin_2), R1.2, R2.2, R3.2, R4.2, R13.2, R14.2, R15.2, R16.2
- net at J2.11 (Pin_11), R3.1: now also R11.2; no longer U1.15 (X2)
- net at J2.13 (Pin_13), R2.1: now also R10.2; no longer U1.14 (X1)
- net at J2.15 (Pin_15), R1.1: now also R9.2; no longer U1.13 (X0)
- net at J2.9 (Pin_9), R4.1: now also R12.2; no longer U1.12 (X3)
- net at U1.1 (X4): now also R13.1
- net at U1.2 (X6): now also R15.1
- net at U1.4 (X7): now also R16.1
- net at U1.5 (X5): now also R14.1
- net at J1.5 (Pin_5), U1.9 (C): now also U1.6 (Inh)
- new net: R9.1, U1.13 (X0)
- new net: R10.1, U1.14 (X1)
- new net: R11.1, U1.15 (X2)
- new net: R12.1, U1.12 (X3)
- no-connect marks 12 -> 0
Other:
- moved on the sheet: C2, J2, J3, R1, R2, R3, R4, U1
