File: Circuit/terminal7/terminal7.sch (KiCad schematic (older format))
At the start: 13 parts, among them J1 Conn_01x05_Male, J2 Conn_02x08_Odd_Even, J3 Conn_01x02_Male, U1 4051

Commit message: ECM対策
Parts:
- removed R7: 10k, Resistor_THT:R_Axial_DIN0204_L3.6mm_D1.6mm_P7.62mm_Horizontal, symbol Device:R
- added R10, R11, R12, R13, R14, R15, R16, R9: 220, Resistor_THT:R_Axial_DIN0204_L3.6mm_D1.6mm_P7.62mm_Horizontal, symbol Device:R
Connections:
- net at J2.1 (Pin_1): now also R16.2; no longer U1.4 (X7)
- net at J2.10 (Pin_10), J2.12 (Pin_12), J2.14 (Pin_14)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: now also J2.3 (Pin_3), R15.2
- net at J2.11 (Pin_11), R3.1: now also R11.2; no longer U1.15 (X2)
- net at J2.13 (Pin_13), R2.1: now also R10.2; no longer U1.14 (X1)
- net at J2.15 (Pin_15), R1.1: now also R9.2; no longer U1.13 (X0)
- net at U1.2 (X6): now also R15.1; no longer J2.3 (Pin_3)
- net at J2.5 (Pin_5), R6.1: now also R14.2; no longer U1.5 (X5)
- net at J2.7 (Pin_7), R5.1: now also R13.2; no longer U1.1 (X4)
- net at J2.9 (Pin_9), R4.1: now also R12.2; no longer U1.12 (X3)
- new net: R9.1, U1.13 (X0)
- new net: R10.1, U1.14 (X1)
- new net: R11.1, U1.15 (X2)
- new net: R12.1, U1.12 (X3)
- new net: R13.1, U1.1 (X4)
- new net: R14.1, U1.5 (X5)
- new net: R16.1, U1.4 (X7)
Other:
- moved on the sheet: C2, J3, U1
Changed lines of the file:
@@
 L 4xxx:4051 U1
 U 1 1 60481B08
-P 4850 2950
-F 0 "U1" H 5394 2996 50  0000 L CNN
-F 1 "4051" H 5394 2905 50  0000 L CNN
-F 2 "Package_DIP:DIP-16_W7.62mm" H 4850 2950 50  0001 C CNN
-F 3 "http://www.intersil.com/content/dam/Intersil/documents/cd40/cd4051bms-52bms-53bms.pdf" H 4850 2950 50  0001 C CNN
-	1    4850 2950
-	1    0    0    -1
-$EndComp
-Wire Wire Line
-	4350 3250 4250 3250
-Wire Wire Line
-	4250 3850 4850 3850
-Connection ~ 4850 3850
-Wire Wire Line
-	4850 3850 4950 3850
+P 5350 2950
+F 0 "U1" H 5894 2996 50  0000 L CNN
+F 1 "4051" H 5894 2905 50  0000 L CNN
+F 2 "Package_DIP:DIP-16_W7.62mm" H 5350 2950 50  0001 C CNN
+F 3 "http://www.intersil.com/content/dam/Intersil/documents/cd40/cd4051bms-52bms-53bms.pdf" H 5350 2950 50  0001 C CNN
+	1    5350 2950
+	1    0    0    -1
+$EndComp
+Connection ~ 5350 3850
+Wire Wire Line
+	5350 3850 5450 3850
 $Comp
 L power:GND #PWR03
@@
 	1    0    0    -1
 $EndComp
-Connection ~ 4250 3850
 $Comp
 L Device:C C2
 U 1 1 604831DD
-P 4700 1950
-F 0 "C2" V 4448 1950 50  0000 C CNN
-F 1 "0.1u" V 4539 1950 50  0000 C CNN
-F 2 "Capacitor_THT:C_Disc_D3.0mm_W1.6mm_P2.50mm" H 4738 1800 50  0001 C CNN
-F 3 "~" H 4700 1950 50  0001 C CNN
-	1    4700 1950
+P 5200 1950
+F 0 "C2" V 4948 1950 50  0000 C CNN
+F 1 "0.1u" V 5039 1950 50  0000 C CNN
+F 2 "Capacitor_THT:C_Disc_D3.0mm_W1.6mm_P2.50mm" H 5238 1800 50  0001 C CNN
+F 3 "~" H 5200 1950 50  0001 C CNN
+	1    5200 1950
 	0    1    1    0
 $EndComp
@@
 $EndComp
 Wire Wire Line
-	4850 1950 4850 2050
+	5350 1950 5350 2050
 $Comp
 L power:GND #PWR04
 U 1 1 6048C611
-P 4550 1950
-F 0 "#PWR04" H 4550 1700 50  0001 C CNN
-F 1 "GND" H 4555 1777 50  0000 C CNN
-F 2 "" H 4550 1950 50  0001 C CNN
-F 3 "" H 4550 1950 50  0001 C CNN
-	1    4550 1950
+P 5050 1950
+F 0 "#PWR04" H 5050 1700 50  0001 C CNN
+F 1 "GND" H 5055 1777 50  0000 C CNN
+F 2 "" H 5050 1950 50  0001 C CNN
+F 3 "" H 5050 1950 50  0001 C CNN
+	1    5050 1950
 	1    0    0    -1
 $EndComp
@@
 	0    1    1    0
 $EndComp
-$Comp
-L Device:R R7
-U 1 1 604ABA9A
-P 3450 3000
-F 0 "R7" V 3450 3000 50  0000 C CNN
-F 1 "10k" V 3400 3200 50  0000 C CNN
-F 2 "Resistor_THT:R_Axial_DIN0204_L3.6mm_D1.6mm_P7.62mm_Horizontal" V 3380 3000 50  0001 C CNN
-F 3 "~" H 3450 3000 50  0001 C CNN
-	1    3450 3000
-	0    1    1    0
-$EndComp
-Wire Wire Line
-	1900 3350 4350 3350
-Wire Wire Line
-	1900 3450 4350 3450
-Wire Wire Line
-	1900 3550 4350 3550
 Wire Wire Line
 	3600 2400 4350 2400
 Wire Wire Line
 	4350 2400 4350 2350
-Connection ~ 4350 2350
 Wire Wire Line
 	4350 2450 4350 2500
 Wire Wire Line
 	4350 2500 3600 2500
-Connection ~ 4350 2450
 Wire Wire Line
 	3600 2600 4350 2600
 Wire Wire Line
 	4350 2600 4350 2550
-Connection ~ 4350 2550
 Wire Wire Line
 	4350 2650 4350 2700
 Wire Wire Line
 	4350 2700 3600 2700
-Connection ~ 4350 2650
 Wire Wire Line
 	3600 2800 4350 2800
 Wire Wire Line
 	4350 2800 4350 2750
-Connection ~ 4350 2750
 Wire Wire Line
 	4350 2850 4350 2900
 Wire Wire Line
 	4350 2900 3600 2900
-Connection ~ 4350 2850
-Wire Wire Line
-	3600 3000 4350 3000
 Wire Wire Line
 	4350 3000 4350 2950
-Connection ~ 4350 2950
 Wire Wire Line
 	3300 2400 3300 2500
@@
 	3300 2800 3300 2900
 Connection ~ 3300 2900
-Wire Wire Line
-	3300 2900 3300 3000
 Connection ~ 3850 2450
 Wire Wire Line
@@
 L Connector:Conn_01x02_Male J3
 U 1 1 604C548C
-P 5550 2350
-F 0 "J3" H 5522 2232 50  0000 R CNN
-F 1 "Conn_01x02_Male" H 5522 2323 50  0000 R CNN
-F 2 "Connector_PinHeader_2.54mm:PinHeader_1x02_P2.54mm_Horizontal" H 5550 2350 50  0001 C CNN
-F 3 "~" H 5550 2350 50  0001 C CNN
-	1    5550 2350
+P 6050 2350
+F 0 "J3" H 6022 2232 50  0000 R CNN
+F 1 "Conn_01x02_Male" H 6022 2323 50  0000 R CNN
+F 2 "Connector_PinHeader_2.54mm:PinHeader_1x02_P2.54mm_Horizontal" H 6050 2350 50  0001 C CNN
+F 3 "~" H 6050 2350 50  0001 C CNN
+	1    6050 2350
 	-1   0    0    1
 $EndComp
@@
 	3300 2150 3300 1500
 Wire Wire Line
-	3300 1500 5350 1500
-Wire Wire Line
-	5350 1500 5350 2250
+	5850 1500 5850 2250
 Connection ~ 3300 2150
 $Comp
 L power:VDD #PWR05
 U 1 1 604CE1F8
-P 4850 1950
-F 0 "#PWR05" H 4850 1800 50  0001 C CNN
-F 1 "VDD" H 4865 2123 50  0000 C CNN
-F 2 "" H 4850 1950 50  0001 C CNN
-F 3 "" H 4850 1950 50  0001 C CNN
-	1    4850 1950
-	1    0    0    -1
-$EndComp
-Connection ~ 4850 1950
+P 5350 1950
+F 0 "#PWR05" H 5350 1800 50  0001 C CNN
+F 1 "VDD" H 5365 2123 50  0000 C CNN
+F 2 "" H 5350 1950 50  0001 C CNN
+F 3 "" H 5350 1950 50  0001 C CNN
+	1    5350 1950
+	1    0    0    -1
+$EndComp
+Connection ~ 5350 1950
 $Comp
 L power:PWR_FLAG #FLG02
@@
 	3850 2150 3850 2350
 Connection ~ 3850 2350
+Wire Wire Line
+	3300 1500 5850 1500
+$Comp
+L Device:R R9
+U 1 1 6041C195
+P 4600 2350
+F 0 "R9" V 4600 2350 50  0000 C CNN
+F 1 "220" V 4550 2550 50  0000 C CNN
+F 2 "Resistor_THT:R_Axial_DIN0204_L3.6mm_D1.6mm_P7.62mm_Horizontal" V 4530 2350 50  0001 C CNN
+F 3 "~" H 4600 2350 50  0001 C CNN
+	1    4600 2350
+	0    1    1    0
+$EndComp
+Wire Wire Line
+	4350 2350 4450 2350
+Connection ~ 4350 2350
+Wire Wire Line
+	4750 2350 4850 2350
+$Comp
+L Device:R R10
+U 1 1 60427657
+P 4600 2450
+F 0 "R10" V 4600 2450 50  0000 C CNN
+F 1 "220" V 4550 2650 50  0000 C CNN
+F 2 "Resistor_THT:R_Axial_DIN0204_L3.6mm_D1.6mm_P7.62mm_Horizontal" V 4530 2450 50  0001 C CNN
+F 3 "~" H 4600 2450 50  0001 C CNN
+	1    4600 2450
+	0    1    1    0
+$EndComp
+$Comp
+L Device:R R11
+U 1 1 60427859
+P 4600 2550
+F 0 "R11" V 4600 2550 50  0000 C CNN
+F 1 "220" V 4550 2750 50  0000 C CNN
+F 2 "Resistor_THT:R_Axial_DIN0204_L3.6mm_D1.6mm_P7.62mm_Horizontal" V 4530 2550 50  0001 C CNN
+F 3 "~" H 4600 2550 50  0001 C CNN
+	1    4600 2550
+	0    1    1    0
+$EndComp
+$Comp
+L Device:R R12
+U 1 1 60427A23
+P 4600 2650
+F 0 "R12" V 4600 2650 50  0000 C CNN
+F 1 "220" V 4550 2850 50  0000 C CNN
+F 2 "Resistor_THT:R_Axial_DIN0204_L3.6mm_D1.6mm_P7.62mm_Horizontal" V 4530 2650 50  0001 C CNN
+F 3 "~" H 4600 2650 50  0001 C CNN
+	1    4600 2650
+	0    1    1    0
+$EndComp
+$Comp
+L Device:R R13
+U 1 1 60427BF9
+P 4600 2750
+F 0 "R13" V 4600 2750 50  0000 C CNN
+F 1 "220" V 4550 2950 50  0000 C CNN
+F 2 "Resistor_THT:R_Axial_DIN0204_L3.6mm_D1.6mm_P7.62mm_Horizontal" V 4530 2750 50  0001 C CNN
+F 3 "~" H 4600 2750 50  0001 C CNN
+	1    4600 2750
+	0    1    1    0
+$EndComp
+$Comp
+L Device:R R14
+U 1 1 60427DEB
+P 4600 2850
+F 0 "R14" V 4600 2850 50  0000 C CNN
+F 1 "220" V 4550 3050 50  0000 C CNN
+F 2 "Resistor_THT:R_Axial_DIN0204_L3.6mm_D1.6mm_P7.62mm_Horizontal" V 4530 2850 50  0001 C CNN
+F 3 "~" H 4600 2850 50  0001 C CNN
+	1    4600 2850
+	0    1    1    0
+$EndComp
+$Comp
+L Device:R R15
+U 1 1 60427FD9
+P 4600 2950
+F 0 "R15" V 4600 2950 50  0000 C CNN
+F 1 "220" V 4550 3150 50  0000 C CNN
+F 2 "Resistor_THT:R_Axial_DIN0204_L3.6mm_D1.6mm_P7.62mm_Horizontal" V 4530 2950 50  0001 C CNN
+F 3 "~" H 4600 2950 50  0001 C CNN
+	1    4600 2950
+	0    1    1    0
+$EndComp
+$Comp
+L Device:R R16
+U 1 1 604281E3
+P 4600 3050
+F 0 "R16" V 4600 3050 50  0000 C CNN
+F 1 "220" V 4550 3250 50  0000 C CNN
+F 2 "Resistor_THT:R_Axial_DIN0204_L3.6mm_D1.6mm_P7.62mm_Horizontal" V 4530 3050 50  0001 C CNN
+F 3 "~" H 4600 3050 50  0001 C CNN
+	1    4600 3050
+	0    1    1    0
+$EndComp
+Wire Wire Line
+	4350 2450 4450 2450
+Connection ~ 4350 2450
+Wire Wire Line
+	4350 2550 4450 2550
+Connection ~ 4350 2550
+Wire Wire Line
+	4350 2650 4450 2650
+Connection ~ 4350 2650
+Wire Wire Line
+	4450 2750 4350 2750
+Connection ~ 4350 2750
+Wire Wire Line
+	4350 2850 4450 2850
+Connection ~ 4350 2850
+Wire Wire Line
+	4450 2950 4350 2950
+Connection ~ 4350 2950
+Wire Wire Line
+	4350 3050 4450 3050
+Wire Wire Line
+	4750 3050 4850 3050
+Wire Wire Line
+	4850 2950 4750 2950
+Wire Wire Line
+	4750 2850 4850 2850
+Wire Wire Line
+	4850 2750 4750 2750
+Wire Wire Line
+	4750 2650 4850 2650
+Wire Wire Line
+	4850 2550 4750 2550
+Wire Wire Line
+	4750 2450 4850 2450
+Wire Wire Line
+	4250 3250 4850 3250
+Wire Wire Line
+	1900 3350 4850 3350
+Wire Wire Line
+	1900 3450 4850 3450
+Wire Wire Line
+	1900 3550 4850 3550
+Wire Wire Line
+	4250 3850 5350 3850
+Connection ~ 4250 3850
+Wire Wire Line
+	3300 2900 3300 3000
+Wire Wire Line
+	4350 3000 3300 3000
 $Comp
 L power:VDD #PWR?
-U 1 1 60375FF5
-P 3100 3050
-F 0 "#PWR?" H 3100 2900 50  0001 C CNN
-F 1 "VDD" H 3115 3223 50  0000 C CNN
-F 2 "" H 3100 3050 50  0001 C CNN
-F 3 "" H 3100 3050 50  0001 C CNN
-	1    3100 3050
-	1    0    0    -1
-$EndComp
-Wire Wire Line
-	3850 3050 3100 3050
+U 1 1 60416052
+P 3150 3050
+F 0 "#PWR?" H 3150 2900 50  0001 C CNN
+F 1 "VDD" H 3165 3223 50  0000 C CNN
+F 2 "" H 3150 3050 50  0001 C CNN
+F 3 "" H 3150 3050 50  0001 C CNN
+	1    3150 3050
+	1    0    0    -1
+$EndComp
+Wire Wire Line
+	3850 3050 3150 3050
 $EndSCHEMATC
