File: Circuit/terminal8(fader)/fader.kicad_pcb (KiCad board)
At the start: 2 copper layers, 24 parts, among them J1 Conn_01x05_Male, J2 0.1u, J3 Conn_01x02_Male, U1 4051

Commit message: ECM対策
Other:
- board outline added: 45.7 x 71.1 mm
- board text added: "Akizuki Type C Board (17x27)"
