File: Circuit/Mother/Mother.kicad_pcb (KiCad board)
At the start: 4 copper layers, 29 parts, among them J1 Conn_PIC_ICSP_ICD, J2 Conn_01x04_Female, U1 TBD62783A, U2 PIC16F18854-SO, U3 ULN2803A

Commit message: mother回路図作成
Parts:
- removed AFF1, AFF2, AFF3, AFF4, AFF5: LTS-6960HR, Display_7Segment:7SegmentLED_LTS6760_LTS6780
- removed BAR1: HDSP-4830_2, Display:HDSP-4830
- removed D3, D4: LED, LED_THT:LED_D3.0mm
- added C10: 0.1u, Capacitor_THT:C_Disc_D3.0mm_W1.6mm_P2.50mm, F.Cu at (163.8, 113.6)
- added C11: 0.1u, Capacitor_THT:C_Disc_D3.0mm_W1.6mm_P2.50mm, F.Cu at (177.0, 100.0)
- added C12: 0.1u, Capacitor_THT:C_Disc_D3.0mm_W1.6mm_P2.50mm, F.Cu at (159.9, 117.0)
- added C13: 0.1u, Capacitor_THT:C_Disc_D3.0mm_W1.6mm_P2.50mm, F.Cu at (188.3, 88.9)
- added C14: 0.1u, Capacitor_THT:C_Disc_D3.0mm_W1.6mm_P2.50mm, F.Cu at (188.3, 85.8)
- added C15: 0.1u, Capacitor_THT:C_Disc_D3.0mm_W1.6mm_P2.50mm, F.Cu at (171.3, 105.5)
- added C16: 0.1u, Capacitor_THT:C_Disc_D3.0mm_W1.6mm_P2.50mm, F.Cu at (165.7, 102.6)
- added C17: 0.1u, Capacitor_THT:C_Disc_D3.0mm_W1.6mm_P2.50mm, F.Cu at (176.5, 96.8)
- added C18: 0.1u, Capacitor_THT:C_Disc_D3.0mm_W1.6mm_P2.50mm, F.Cu at (160.0, 102.6)
- added C19: 0.1u, Capacitor_THT:C_Disc_D3.0mm_W1.6mm_P2.50mm, F.Cu at (165.6, 105.8)
- added C20: 0.1u, Capacitor_THT:C_Disc_D3.0mm_W1.6mm_P2.50mm, F.Cu at (182.6, 87.1)
- added C21: 10u, Capacitor_THT:CP_Radial_D5.0mm_P2.50mm, F.Cu at (179.2, 92.0)
- added C22: 10uF, Capacitor_THT:C_Disc_D5.0mm_W2.5mm_P5.00mm, F.Cu at (157.5, 106.9)
- added C5: 0.1u, Capacitor_THT:C_Disc_D3.0mm_W1.6mm_P2.50mm, F.Cu at (171.3, 102.4)
- added C6: 0.1u, Capacitor_THT:C_Disc_D3.0mm_W1.6mm_P2.50mm, F.Cu at (169.5, 108.9)
- added C7: 10u, Capacitor_THT:CP_Radial_D5.0mm_P2.50mm, F.Cu at (172.6, 92.0)
- added C8: 0.1u, Capacitor_THT:C_Disc_D3.0mm_W1.6mm_P2.50mm, F.Cu at (182.2, 96.8)
- added C9: 10u, Capacitor_THT:CP_Radial_D5.0mm_P2.50mm, F.Cu at (186.3, 80.9)
- added F1: RXEF050, Capacitor_THT:C_Disc_D8.0mm_W2.5mm_P5.00mm, F.Cu at (186.4, 71.8)
- added J3: Conn_02x09_Odd_Even, Connector_PinHeader_2.54mm:PinHeader_2x09_P2.54mm_Horizontal, F.Cu at (128.5, 72.1)
- added J4: Conn_01x04_Male, Connector_PinHeader_2.54mm:PinHeader_1x04_P2.54mm_Horizontal, F.Cu at (162.5, 72.1)
- added J5: Conn_02x09_Odd_Even, Connector_PinHeader_2.54mm:PinHeader_2x09_P2.54mm_Horizontal, F.Cu at (112.6, 72.1)
- added J6: Conn_PIC_ICSP_ICD, Connector_PinHeader_2.54mm:PinHeader_1x06_P2.54mm_Vertical, F.Cu at (144.5, 72.1)
- added J7: Conn_01x05_Male, Connector_PinHeader_2.54mm:PinHeader_1x05_P2.54mm_Horizontal, F.Cu at (149.1, 72.1)
- added R11: 10k, Resistor_THT:R_Axial_DIN0204_L3.6mm_D1.6mm_P7.62mm_Horizontal, F.Cu at (159.9, 96.3)
- added R12: 10k, Resistor_THT:R_Axial_DIN0204_L3.6mm_D1.6mm_P7.62mm_Horizontal, F.Cu at (175.1, 80.8)
- added R13: 10k, Resistor_THT:R_Axial_DIN0204_L3.6mm_D1.6mm_P7.62mm_Horizontal, F.Cu at (161.4, 93.1)
- added R14: 10k, Resistor_THT:R_Axial_DIN0204_L3.6mm_D1.6mm_P7.62mm_Horizontal, F.Cu at (159.9, 99.5)
- added R15: 10k, Resistor_THT:R_Axial_DIN0204_L3.6mm_D1.6mm_P7.62mm_Horizontal, F.Cu at (111.4, 118.2)
- added R16: 10k, Resistor_THT:R_Axial_DIN0204_L3.6mm_D1.6mm_P7.62mm_Horizontal, F.Cu at (172.0, 87.1)
- added R17: 10k, Resistor_THT:R_Axial_DIN0204_L3.6mm_D1.6mm_P7.62mm_Horizontal, F.Cu at (172.2, 84.0)
- added R18: 10k, Resistor_THT:R_Axial_DIN0204_L3.6mm_D1.6mm_P7.62mm_Horizontal, F.Cu at (146.5, 114.3)
- added R19: 10k, Resistor_THT:R_Axial_DIN0204_L3.6mm_D1.6mm_P7.62mm_Horizontal, F.Cu at (136.0, 120.6)
- added R20: 220, Resistor_THT:R_Axial_DIN0204_L3.6mm_D1.6mm_P7.62mm_Horizontal, F.Cu at (161.4, 86.8)
- added R21: 220, Resistor_THT:R_Axial_DIN0204_L3.6mm_D1.6mm_P7.62mm_Horizontal, F.Cu at (144.0, 111.1)
- added R22: 220, Resistor_THT:R_Axial_DIN0204_L3.6mm_D1.6mm_P7.62mm_Horizontal, F.Cu at (175.1, 74.5)
- added R23: 220, Resistor_THT:R_Axial_DIN0204_L3.6mm_D1.6mm_P7.62mm_Horizontal, F.Cu at (136.0, 114.3)
- added U4: PIC32MX110F016B-I_SP, Package_DIP:DIP-28_W7.62mm, F.Cu at (101.0, 71.9)
- added U5: 4051, Package_DIP:DIP-16_W7.62mm, F.Cu at (111.9, 96.8)
- added U6: TLP785, Package_DIP:DIP-4_W7.62mm, F.Cu at (101.0, 109.0)
- C2: value 0.1u -> 10u; footprint Capacitor_THT:C_Disc_D3.0mm_W1.6mm_P2.50mm -> Capacitor_THT:CP_Radial_D5.0mm_P2.50mm
- C3: value 0.01u -> 10u; footprint Capacitor_THT:C_Disc_D3.0mm_W2.0mm_P2.50mm -> Capacitor_THT:CP_Radial_D5.0mm_P2.50mm
- D2: value LED -> 1SS178; footprint LED_THT:LED_D3.0mm -> Diode_THT:D_DO-35_SOD27_P3.81mm_Vertical_AnodeUp
- J1: value Conn_PIC_ICSP_ICD -> Conn_01x02_Male; footprint Connector_PinHeader_2.54mm:PinHeader_1x06_P2.54mm_Vertical -> Connector_PinHeader_2.54mm:PinHeader_1x02_P2.54mm_Horizontal
- J2: value Conn_01x04_Female -> Conn_01x05_Male; footprint Connector_PinSocket_2.54mm:PinSocket_1x04_P2.54mm_Vertical -> Connector_PinHeader_2.54mm:PinHeader_1x05_P2.54mm_Horizontal
- R1, R3: value 4.7k -> 1k
- R10, R2, R4, R5, R6, R7, R9: value 4.7k -> 10k
- U1: value TBD62783A -> 74HC00; footprint Package_DIP:DIP-18_W7.62mm -> Package_DIP:DIP-14_W7.62mm
- U2: value PIC16F18854-SO -> BP5293-33; footprint Package_DIP:DIP-28_W7.62mm -> Converter_DCDC:Converter_DCDC_RECOM_R-78B-2.0_THT
- U3: value ULN2803A -> BP5293-50; footprint Package_DIP:DIP-18_W7.62mm -> Converter_DCDC:Converter_DCDC_RECOM_R-78B-2.0_THT
- moved R10 98.1 mm to (175.1, 77.7)
- moved D1 93.8 mm to (170.7, 98.0), turned to 0 degrees
- moved R5 86.1 mm to (175.1, 71.4), turned to 0 degrees
- moved R9 68.5 mm to (161.4, 89.9)
- moved R4 65.9 mm to (161.7, 83.6), turned to 0 degrees
- moved C4 61.2 mm to (153.8, 119.1), turned to 0 degrees
- moved R7 55.6 mm to (146.8, 106.4), turned to 0 degrees
- moved J2 53.3 mm to (134.3, 97.1), turned to 0 degrees
- moved D2 50.4 mm to (186.0, 75.7), turned to 0 degrees
- moved C1 47.9 mm to (163.8, 110.5), turned to 0 degrees
- moved R6 42.8 mm to (136.0, 117.4), turned to 0 degrees
- moved J1 35.2 mm to (123.4, 116.5)
- moved R2 31.7 mm to (133.4, 111.1), turned to 0 degrees
- moved U1 27.8 mm to (122.7, 96.8), turned to 0 degrees
- moved C3 27.4 mm to (157.7, 112.2), turned to 0 degrees
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Connections:
- C1 pad 1: VDD -> GND
- C1 pad 2: GND -> +5V
- C2 pad 1: GND -> Net-(C2-Pad1)
- C2 pad 2: VDD -> GND
- C3 pad 1: GND -> Net-(C2-Pad1)
- C3 pad 2: VDD -> GND
- C4 pad 1: GND -> Net-(C4-Pad1)
- C4 pad 2: VDD -> GND
- D1 pad 1: /LED_D6 -> GND
- D1 pad 2: /LED_S3 -> Net-(C4-Pad1)
- D2 pad 1: /LED_D6 -> Net-(D2-Pad1)
- D2 pad 2: /LED_S4 -> Net-(D2-Pad2)
- J1 pad 1: Net-(J1-Pad1) -> Net-(F1-Pad2)
- J1 pad 2: VDD -> GND
- J2 pad 4: GND -> Net-(J2-Pad4)
- R1 pad 1: /LED_S0 -> VDD
- R1 pad 2: Net-(R1-Pad2) -> Net-(C4-Pad1)
- R10 pad 2: Net-(J2-Pad2) -> Net-(J3-Pad15)
- R2 pad 1: /LED_S1 -> VDD
- R2 pad 2: Net-(R2-Pad2) -> Net-(C6-Pad2)
- R3 pad 1: /LED_S2 -> Net-(C6-Pad2)
- R3 pad 2: Net-(R3-Pad2) -> Net-(J6-Pad1)
- R4 pad 1: /LED_S3 -> VDD
- R4 pad 2: Net-(R4-Pad2) -> Net-(J3-Pad3)
- R5 pad 1: /LED_S4 -> VDD
- R5 pad 2: Net-(R5-Pad2) -> Net-(J3-Pad5)
- R6 pad 1: /LED_S5 -> VDD
- R6 pad 2: Net-(R6-Pad2) -> Net-(J3-Pad7)
- R7 pad 1: /LED_S6 -> VDD
- R7 pad 2: Net-(R7-Pad2) -> Net-(J3-Pad10)
- R8 pad 2: Net-(J1-Pad1) -> Net-(J3-Pad11)
- R9 pad 2: Net-(J2-Pad3) -> Net-(J3-Pad13)
- U1 pad 11: Net-(R1-Pad2) -> (no net)
- U1 pad 12: Net-(R2-Pad2) -> GND
- U1 pad 13: Net-(R3-Pad2) -> GND
- U1 pad 14: Net-(R4-Pad2) -> +5V
- U1 pad 2: Net-(U1-Pad2) -> Net-(U1-Pad1)
- U1 pad 4: Net-(U1-Pad4) -> Net-(U1-Pad3)
- U1 pad 5: Net-(U1-Pad5) -> Net-(U1-Pad3)
- U1 pad 6: Net-(U1-Pad6) -> Net-(R22-Pad1)
- U1 pad 7: Net-(U1-Pad7) -> GND
- U1 pad 8: Net-(U1-Pad8) -> (no net)
- U1 pad 9: VDD -> GND
- U2 pad 1: Net-(J1-Pad1) -> Net-(C2-Pad1)
- U2 pad 2: Net-(U1-Pad8) -> GND
- U2 pad 3: Net-(U1-Pad7) -> VDD
- U3 pad 1: Net-(U2-Pad26) -> Net-(C2-Pad1)
- U3 pad 2: Net-(U2-Pad25) -> GND
- U3 pad 3: Net-(U2-Pad24) -> +5V
Routing:
- net /LED_S1: track 188.0 -> 0.00 mm, vias 9 -> 0
- net /LED_S6: track 184.1 -> 0.00 mm, vias 8 -> 0
- net /LED_S5: track 178.0 -> 0.00 mm, vias 8 -> 0
- net /LED_S4: track 173.8 -> 0.00 mm, vias 9 -> 0
- net /LED_S3: track 171.2 -> 0.00 mm, vias 8 -> 0
- net /LED_S0: track 167.6 -> 0.00 mm, vias 9 -> 0
- net /LED_D6: track 153.7 -> 0.00 mm, vias 1 -> 0
- net GND: track 148.2 -> 0.00 mm, vias 2 -> 0
- net /LED_S2: track 147.3 -> 0.00 mm, vias 6 -> 0
- net VDD: track 125.8 -> 0.00 mm, vias 3 -> 0
- net /LED_D4: track 86.9 -> 0.00 mm
- net /LED_D3: track 62.8 -> 0.00 mm
- net /LED_D0: track 61.9 -> 0.00 mm
- net /LED_D5: track 54.8 -> 0.00 mm
- net /LED_D2: track 51.7 -> 0.00 mm
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
Commit message: 基板完成
Parts:
- removed C13: 0.1u, Capacitor_THT:C_Disc_D3.0mm_W1.6mm_P2.50mm
- C21: footprint Capacitor_THT:CP_Radial_D5.0mm_P2.50mm -> Capacitor_THT:C_Axial_L5.1mm_D3.1mm_P7.50mm_Horizontal
- D2: footprint Diode_THT:D_DO-35_SOD27_P3.81mm_Vertical_AnodeUp -> Diode_THT:D_DO-35_SOD27_P2.54mm_Vertical_AnodeUp
- J6: footprint Connector_PinHeader_2.54mm:PinHeader_1x06_P2.54mm_Vertical -> Connector_PinHeader_2.54mm:PinHeader_1x06_P2.54mm_Horizontal
- U2, U3: footprint Converter_DCDC:Converter_DCDC_RECOM_R-78B-2.0_THT -> Package_TO_SOT_THT:TO-220-3_Vertical
- moved F1 95.5 mm to (116.8, 137.2), turned to 180 degrees
- moved R8 92.2 mm to (180.3, 68.6), turned to 180 degrees
- moved J4 78.3 mm to (106.7, 127.0), turned to 180 degrees
- moved R3 77.9 mm to (188.0, 106.7), turned to 180 degrees
- moved C21 76.0 mm to (111.8, 127.0), turned to 90 degrees
- moved U4 75.2 mm to (167.6, 106.7), turned to 270 degrees
- moved D2 69.8 mm to (119.4, 96.5), turned to 270 degrees
- moved R15 67.7 mm to (160.0, 71.1), turned to 180 degrees
- moved R22 66.5 mm to (116.8, 106.7), turned to 180 degrees
- moved J5 65.9 mm to (177.8, 81.3)
- moved R6 62.3 mm to (180.3, 73.7), turned to 180 degrees
- moved R19 61.2 mm to (149.9, 61.0), turned to 180 degrees
- moved C7 61.0 mm to (111.8, 87.6), turned to 90 degrees
- moved J6 55.4 mm to (180.3, 114.3)
- moved J7 54.7 mm to (106.7, 106.7), turned to 180 degrees
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Connections:
- U4 pad 2: Net-(J5-Pad1) -> Net-(J5-Pad17)
- U4 pad 24: Net-(J5-Pad17) -> Net-(J5-Pad1)
- U4 pad 25: Net-(J5-Pad15) -> Net-(J5-Pad3)
- U4 pad 26: Net-(J5-Pad13) -> Net-(J5-Pad5)
- U4 pad 3: Net-(J5-Pad3) -> Net-(J5-Pad15)
- U4 pad 4: Net-(J5-Pad5) -> Net-(J5-Pad13)
- U4 pad 5: Net-(J5-Pad7) -> Net-(J5-Pad11)
- U4 pad 7: Net-(J5-Pad11) -> Net-(J5-Pad7)
Routing:
- net GND: track 0.00 -> 413.4 mm, vias 0 -> 6
- net VDD: track 0.00 -> 279.4 mm, vias 0 -> 10
- net Net-(C4-Pad1): track 0.00 -> 99.1 mm
- net Net-(J2-Pad2): track 0.00 -> 64.9 mm, vias 0 -> 2
- net Net-(J2-Pad3): track 0.00 -> 59.8 mm, vias 0 -> 2
- net Net-(J2-Pad4): track 0.00 -> 55.9 mm, vias 0 -> 2
- net Net-(U4-Pad23): track 0.00 -> 55.2 mm
- net Net-(J5-Pad1): track 0.00 -> 53.3 mm, vias 0 -> 2
- net Net-(J5-Pad5): track 0.00 -> 53.3 mm, vias 0 -> 2
- net Net-(J5-Pad3): track 0.00 -> 48.3 mm, vias 0 -> 2
- net Net-(J4-Pad2): track 0.00 -> 46.8 mm
- net Net-(C20-Pad2): track 0.00 -> 43.2 mm
- net Net-(C16-Pad2): track 0.00 -> 43.2 mm
- net Net-(C18-Pad2): track 0.00 -> 40.7 mm, vias 0 -> 2
- net Net-(J4-Pad3): track 0.00 -> 39.2 mm
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Other:
- board text added: "34x35"

Commit message: 回路系全完成
Parts:
- added D3: 1N4007, Diode_THT:D_DO-41_SOD81_P2.54mm_Vertical_AnodeUp, F.Cu at (109.2, 137.2)
- moved J1 2.54 mm to (104.1, 137.2)
Connections:
- F1 pad 2: Net-(F1-Pad2) -> Net-(D3-Pad1)
- J1 pad 1: Net-(F1-Pad2) -> Net-(D3-Pad2)
- R23 pad 1: GND -> VDD
Routing:
- net VDD: track 279.4 -> 299.5 mm, vias 10 -> 12
- net Net-(F1-Pad2): track 5.08 -> 0.00 mm
- net Net-(D3-Pad2): track 0.00 -> 2.54 mm
- net Net-(D3-Pad1): track 0.00 -> 2.54 mm
