File: Circuit/Mother/Mother.kicad_pcb (KiCad board)
At the start: 4 copper layers, 57 parts, among them J1 Conn_01x02_Male, J2 Conn_01x05_Male, J3 Conn_02x09_Odd_Even, J4 Conn_01x04_Male, J5 Conn_02x09_Odd_Even, J6 Conn_PIC_ICSP_ICD, J7 Conn_01x05_Male, U1 74HC00, U2 BP5293-33, U3 BP5293-50, U4 PIC32MX110F016B-I_SP, U5 4051, U6 TLP785

Commit message: メイン飛んだ
Parts:
- added C20: 0.1u, Capacitor_THT:C_Disc_D3.0mm_W1.6mm_P2.50mm, F.Cu at (170.2, 167.6)
- added C21: 0.01u, Capacitor_THT:C_Disc_D3.0mm_W2.0mm_P2.50mm, F.Cu at (167.6, 167.6)
- added C22: 0.1u, Capacitor_THT:C_Disc_D3.0mm_W1.6mm_P2.50mm, F.Cu at (185.4, 172.7)
- added C23: 0.1u, Capacitor_THT:C_Disc_D3.0mm_W1.6mm_P2.50mm, F.Cu at (106.7, 154.9)
- added C24: 10u, Capacitor_THT:CP_Radial_D5.0mm_P2.50mm, F.Cu at (160.0, 132.1)
- added C25: 0.1u, Capacitor_THT:C_Disc_D3.0mm_W1.6mm_P2.50mm, F.Cu at (162.6, 134.6)
- added D3: LED, LED_THT:LED_D5.0mm, F.Cu at (167.6, 134.6)
- added J10: Conn_01x07_Female, Connector_PinSocket_2.54mm:PinSocket_1x07_P2.54mm_Vertical, F.Cu at (185.4, 149.9)
- added J11: Conn_02x08_Odd_Even, Connector_PinHeader_2.54mm:PinHeader_2x08_P2.54mm_Horizontal, F.Cu at (96.5, 55.9)
- added J8: Conn_01x07_Female, Connector_PinSocket_2.54mm:PinSocket_1x07_P2.54mm_Vertical, F.Cu at (142.2, 162.6)
- added J9: Conn_PIC_ICSP_ICD, Connector_PinHeader_2.54mm:PinHeader_1x06_P2.54mm_Horizontal, F.Cu at (190.5, 137.2)
- added R23: 10k, Resistor_THT:R_Axial_DIN0204_L3.6mm_D1.6mm_P7.62mm_Horizontal, F.Cu at (149.9, 137.2)
- added R24: 4.7k, Resistor_THT:R_Axial_DIN0204_L3.6mm_D1.6mm_P7.62mm_Horizontal, F.Cu at (147.3, 177.8)
- added R25: 4.7k, Resistor_THT:R_Axial_DIN0204_L3.6mm_D1.6mm_P7.62mm_Horizontal, F.Cu at (175.3, 177.8)
- added R26: 1Meg, Resistor_THT:R_Axial_DIN0204_L3.6mm_D1.6mm_P7.62mm_Horizontal, F.Cu at (114.3, 58.4)
- added R27: 1Meg, Resistor_THT:R_Axial_DIN0204_L3.6mm_D1.6mm_P7.62mm_Horizontal, F.Cu at (111.8, 58.4)
- added R28: 1Meg, Resistor_THT:R_Axial_DIN0204_L3.6mm_D1.6mm_P7.62mm_Horizontal, F.Cu at (109.2, 58.4)
- added R29: 1Meg, Resistor_THT:R_Axial_DIN0204_L3.6mm_D1.6mm_P7.62mm_Horizontal, F.Cu at (106.7, 58.4)
- added R30: 1Meg, Resistor_THT:R_Axial_DIN0204_L3.6mm_D1.6mm_P7.62mm_Horizontal, F.Cu at (104.1, 58.4)
- added R31: 1Meg, Resistor_THT:R_Axial_DIN0204_L3.6mm_D1.6mm_P7.62mm_Horizontal, F.Cu at (101.6, 58.4)
- added R32: 220, Resistor_THT:R_Axial_DIN0204_L3.6mm_D1.6mm_P7.62mm_Horizontal, F.Cu at (116.8, 152.4)
- added R33: 220, Resistor_THT:R_Axial_DIN0204_L3.6mm_D1.6mm_P7.62mm_Horizontal, F.Cu at (114.3, 152.4)
- added R34: 220, Resistor_THT:R_Axial_DIN0204_L3.6mm_D1.6mm_P7.62mm_Horizontal, F.Cu at (111.8, 152.4)
- added R35: 220, Resistor_THT:R_Axial_DIN0204_L3.6mm_D1.6mm_P7.62mm_Horizontal, F.Cu at (119.4, 152.4)
- added R36: 220, Resistor_THT:R_Axial_DIN0204_L3.6mm_D1.6mm_P7.62mm_Horizontal, F.Cu at (101.6, 152.4)
- added R37: 220, Resistor_THT:R_Axial_DIN0204_L3.6mm_D1.6mm_P7.62mm_Horizontal, F.Cu at (94.0, 152.4)
- added R38: 220, Resistor_THT:R_Axial_DIN0204_L3.6mm_D1.6mm_P7.62mm_Horizontal, F.Cu at (99.1, 152.4)
- added R39: 220, Resistor_THT:R_Axial_DIN0204_L3.6mm_D1.6mm_P7.62mm_Horizontal, F.Cu at (96.5, 152.4)
- added R40: 1k, Resistor_THT:R_Axial_DIN0204_L3.6mm_D1.6mm_P7.62mm_Horizontal, F.Cu at (147.3, 132.1)
- added U10: 4051, Package_DIP:DIP-16_W7.62mm, F.Cu at (101.6, 157.5)
- added U7: ULN2803A, Package_DIP:DIP-18_W7.62mm, F.Cu at (154.9, 165.1)
- added U8: PIC16F18854-SO, Package_DIP:DIP-28_W7.62mm, F.Cu at (157.5, 144.8)
- added U9: TBD62783A, Package_DIP:DIP-18_W7.62mm, F.Cu at (172.7, 149.9)
- moved D1 7.62 mm to (116.8, 137.2), turned to 90 degrees
- moved F1 5.08 mm to (111.7, 137.2)
- renumbered C12 to C10, C14 to C11, C15 to C12, C16 to C13, C17 to C14, C18 to C15, C19 to C16, C20 to C17, C21 to C18, C22 to C19, C6 to C4, C7 to C5, C8 to C6, C9 to C7, C10 to C8, C11 to C9, D3 to D1, R2 to R1, R11 to R10, R12 to R11, R13 to R12, R14 to R13, R15 to R14, R16 to R15, R17 to R16, R18 to R17, R19 to R18, R20 to R19, R3 to R2, R21 to R20, R22 to R21, R23 to R22, R4 to R3, R5 to R4, R6 to R5, R7 to R6, R8 to R7, R9 to R8, R10 to R9
Connections:
- net Net-(J2-Pad2) renamed /Sheet60E5A5FF/A
- net Net-(J2-Pad3) renamed /Sheet60E5A5FF/B
- net Net-(J2-Pad4) renamed /Sheet60E5A5FF/C
- net Net-(J4-Pad2) renamed /Sheet60D32BD3/SDA
- net Net-(J4-Pad3) renamed /Sheet60D32BD3/SCL
- net Net-(J5-Pad3) renamed /Sheet60E5A5FF/A+
- C6 pad 2: VDD -> /Sheet60E5A5FF/A-
- C7 pad 1: VDD -> /Sheet60E5A5FF/A-
- D1 pad 1: Net-(D3-Pad1) -> Net-(C2-Pad1)
- D1 pad 2: Net-(D3-Pad2) -> GND
- F1 pad 2: Net-(D3-Pad1) -> Net-(F1-Pad2)
- J1 pad 1: Net-(D3-Pad2) -> Net-(F1-Pad2)
- J5 pad 10: VDD -> /Sheet60E5A5FF/A-
- J5 pad 12: VDD -> /Sheet60E5A5FF/A-
- J5 pad 14: VDD -> /Sheet60E5A5FF/A-
- J5 pad 16: VDD -> /Sheet60E5A5FF/A-
- J5 pad 18: VDD -> /Sheet60E5A5FF/A-
- J5 pad 2: VDD -> /Sheet60E5A5FF/A-
- J5 pad 4: VDD -> /Sheet60E5A5FF/A-
- J5 pad 6: VDD -> /Sheet60E5A5FF/A-
- J5 pad 8: VDD -> /Sheet60E5A5FF/A-
Routing:
- net /Sheet60E5A5FF/A-: track 0.00 -> 295.4 mm, vias 0 -> 1
- net GND: track 413.4 -> 614.1 mm, vias 8 -> 13
- net Net-(J11-Pad9): track 0.00 -> 103.0 mm
- net /Sheet60E5A5FF/C: track 55.9 -> 158.6 mm, vias 2 -> 3
- net /Sheet60E5A5FF/B: track 59.8 -> 162.4 mm, vias 2 -> 3
- net /Sheet60E5A5FF/A: track 64.9 -> 167.4 mm, vias 2 -> 3
- net Net-(J11-Pad5): track 0.00 -> 99.1 mm, vias 0 -> 1
- net Net-(J11-Pad15): track 0.00 -> 90.3 mm
- net Net-(J11-Pad7): track 0.00 -> 90.0 mm, vias 0 -> 1
- net Net-(J11-Pad13): track 0.00 -> 90.0 mm
- net Net-(J11-Pad11): track 0.00 -> 90.0 mm
- net /Sheet60E5A5FF/A+: track 48.3 -> 132.1 mm
- net /Sheet60D32BD3/SDA: track 46.8 -> 129.0 mm, vias 0 -> 1
- net /Sheet60D32BD3/SCL: track 39.2 -> 116.0 mm, vias 0 -> 1
- net Net-(J9-Pad1): track 0.00 -> 40.6 mm
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- added copper zone on B.Cu, net GND
- added copper zone on In2.Cu, net VDD
Other:
- board text removed: "34x35"

Commit message: ディスプレイ単独テスト完了
Routing:
- net VDD: track 444.5 -> 473.6 mm, vias 23 -> 22
- net +5V: track 15.3 -> 20.4 mm, vias 1 -> 2
- net Net-(U1-Pad1): track 18.8 -> 15.2 mm
- net Net-(R19-Pad2): track 23.9 -> 25.4 mm
- net Net-(J6-Pad4): vias 0 -> 2
- net Net-(J11-Pad7): vias 1 -> 0
- net Net-(J11-Pad5): vias 1 -> 2
- net GND: vias 13 -> 12
- added copper zone on B.Cu, net VDD
- removed copper zone on In2.Cu, net VDD
