File: Circuit/Mother/Mother.sch (KiCad schematic (older format))
At the start: 86 parts, among them J1 Conn_PIC_ICSP_ICD, J2 Conn_01x02_Male, J3 Conn_01x05_Male, J4 Conn_02x09_Odd_Even, J5 Conn_02x09_Odd_Even, J6 Conn_PIC_ICSP_ICD, J7 Conn_01x05_Male, U1 TBD62783A, U2 PIC16F18854-SO, U3 ULN2803A, U4 74HC00, U5 BP5293-50, U6 BP5293-33, U7 PIC32MX110F016B-I_SP, U8 4051, U9 TLP785

Commit message: mother回路図作成
Parts:
- removed AFF1, AFF2, AFF3, AFF4, AFF5: LTS-6960HR, Display_7Segment:7SegmentLED_LTS6760_LTS6780, symbol Display_Character:LTS-6960HR
- removed BAR1: HDSP-4830_2, Display:HDSP-4830, symbol LED:HDSP-4830_2
- removed C1, C2: 0.1u, Capacitor_THT:C_Disc_D3.0mm_W1.6mm_P2.50mm, symbol Device:C
- removed C3: 0.01u, Capacitor_THT:C_Disc_D3.0mm_W2.0mm_P2.50mm, symbol Device:C
- removed D1, D2, D3, D4: LED, LED_THT:LED_D3.0mm, symbol Device:LED
- removed J1: Conn_PIC_ICSP_ICD, Connector_PinHeader_2.54mm:PinHeader_1x06_P2.54mm_Vertical, symbol Connector:Conn_PIC_ICSP_ICD
- removed R10, R9: 4.7k, Resistor_THT:R_Axial_DIN0204_L3.6mm_D1.6mm_P7.62mm_Horizontal, symbol Device:R
- removed R11, R2, R3, R4, R5, R6, R7: 220, Resistor_THT:R_Axial_DIN0204_L3.6mm_D1.6mm_P7.62mm_Horizontal, symbol Device:R
- removed R8: 10k, Resistor_THT:R_Axial_DIN0204_L3.6mm_D1.6mm_P7.62mm_Horizontal, symbol Device:R
- removed U1: TBD62783A, Package_DIP:DIP-18_W7.62mm, symbol Transistor_Array:TBD62783A
- removed U2: PIC16F18854-SO, Package_DIP:DIP-28_W7.62mm, symbol MCU_Microchip_PIC16:PIC16F18854-SO
- removed U3: ULN2803A, Package_DIP:DIP-18_W7.62mm, symbol Transistor_Array:ULN2803A
- added C?: 10u, Capacitor_THT:CP_Radial_D5.0mm_P2.50mm, symbol Device:CP
- added J?: Conn_01x04_Male, symbol Connector:Conn_01x04_Male
Connections:
- net GND: now also C?.2, J?.4 (Pin_4)
- net VDD: now also C?.1, J?.1 (Pin_1)
- net at U7.17 (TCK/RPB8/SCL1/CTED10/PMD4/RB8): now also J?.3 (Pin_3)
- net at U7.18 (TDO/RPB9/SDA1/CTED4/PMD3/RB9): now also J?.2 (Pin_2)
- no-connect marks 23 -> 6
Other:
- moved on the sheet: C10, C11, C12, C13, C14, C15, C16, C17, C18, C19, C20, C21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

Commit message: 基板完成
Parts:
- removed C16: 0.1u, Capacitor_THT:C_Disc_D3.0mm_W1.6mm_P2.50mm, symbol Device:C
- C21: renamed from C?; footprint Capacitor_THT:CP_Radial_D5.0mm_P2.50mm -> Capacitor_THT:C_Axial_L5.1mm_D3.1mm_P7.50mm_Horizontal
- D2: renamed from D6; footprint Diode_THT:D_DO-35_SOD27_P3.81mm_Vertical_AnodeUp -> Diode_THT:D_DO-35_SOD27_P2.54mm_Vertical_AnodeUp
- J4: renamed from J?; footprint (none) -> Connector_PinHeader_2.54mm:PinHeader_1x04_P2.54mm_Horizontal
- J6: footprint Connector_PinHeader_2.54mm:PinHeader_1x06_P2.54mm_Vertical -> Connector_PinHeader_2.54mm:PinHeader_1x06_P2.54mm_Horizontal
- U2: renamed from U6; footprint Converter_DCDC:Converter_DCDC_RECOM_R-78B-2.0_THT -> Package_TO_SOT_THT:TO-220-3_Vertical
- U3: renamed from U5; footprint Converter_DCDC:Converter_DCDC_RECOM_R-78B-2.0_THT -> Package_TO_SOT_THT:TO-220-3_Vertical
- renumbered C4 to C1, C13 to C10, C14 to C11, C15 to C12, C17 to C14, C18 to C15, C19 to C16, C20 to C17, C21 to C18, C22 to C19, C5 to C2, C23 to C20, C24 to C22, C6 to C3, C7 to C4, C8 to C5, C11 to C6, C12 to C7, C9 to C8, C10 to C9, D5 to D1, J2 to J1, J3 to J2, J4 to J3, R12 to R1, R20 to R10, R21 to R11, R22 to R12, R23 to R13, R24 to R14, R25 to R15, R26 to R16, R27 to R17, R28 to R18, R29 to R19, R13 to R2, R30 to R20, R31 to R21, R32 to R22, R33 to R23, R1 to R3, R14 to R4, R15 to R5, R16 to R6, R17 to R7, R18 to R8, R19 to R9, U4 to U1, U7 to U4, U8 to U5, U9 to U6
Connections:
- net at U4.2 (VREF+/CVREF+/AN0/C3INC/RPA0/CTED1/RA0): now also J5.17 (Pin_17); no longer J5.1 (Pin_1)
- net at U4.24 (AN11/RPB13/CTPLS/PMRD/RB13): now also J5.1 (Pin_1); no longer J5.17 (Pin_17)
- net at U4.25 (CVREFOUT/AN10/C3INB/RPB14/SCK1/CTED5/PMWR/RB14): now also J5.3 (Pin_3); no longer J5.15 (Pin_15)
- net at U4.26 (AN9/C3INA/RPB15/SCK2/CTED6/PMCS1/RB15): now also J5.5 (Pin_5); no longer J5.13 (Pin_13)
- net at U4.3 (VREF-/CVREF-/AN1/RPA1/CTED2/RA1): now also J5.15 (Pin_15); no longer J5.3 (Pin_3)
- net at U4.4 (PGED1/AN2/C1IND/C2INB/C3IND/RPB0/RB0): now also J5.13 (Pin_13); no longer J5.5 (Pin_5)
- net at U4.5 (PGEC1/AN3/C1INC/C2INA/RPB1/CTED12/RB1): now also J5.11 (Pin_11); no longer J5.7 (Pin_7)
- net at U4.7 (AN5/C1INA/C2INC/RTCC/RPB3/SCL2/RB3): now also J5.7 (Pin_7); no longer J5.11 (Pin_11)

Commit message: 回路系全完成
Parts:
- added D3: 1N4007, Diode_THT:D_DO-41_SOD81_P2.54mm_Vertical_AnodeUp, symbol Diode:1N4007
Connections:
- net GND: no longer R23.1
- net VDD: now also R23.1
- net at F1.2: now also D3.1 (K); no longer J1.1 (Pin_1)
- new net: D3.2 (A), J1.1 (Pin_1)
Other:
- moved on the sheet: J1
Changed lines of the file:
@@
 	0    -1   1    0
-$EndComp
-$Comp
-L power:GND #PWR026
-U 1 1 60B975CF
-P 13650 2600
-F 0 "#PWR026" H 13650 2350 50  0001 C CNN
-F 1 "GND" H 13655 2427 50  0000 C CNN
-F 2 "" H 13650 2600 50  0001 C CNN
-F 3 "" H 13650 2600 50  0001 C CNN
-	1    13650 2600
-	1    0    0    -1
 $EndComp
 Wire Wire Line
@@
 Connection ~ 3600 2600
 Wire Wire Line
-	3200 2700 3200 2900
-Wire Wire Line
 	3600 3550 3200 3550
 Connection ~ 3600 3550
@@
 	3600 2900 3200 2900
 Connection ~ 3600 2900
-Connection ~ 3200 2900
 Wire Wire Line
 	3200 2900 3200 3550
@@
 Connection ~ 6000 5600
 Connection ~ 6500 5800
+Wire Wire Line
+	11450 4100 10700 4100
+Connection ~ 3200 3550
+$Comp
+L Device:Polyfuse F1
+U 1 1 62039685
+P 3000 2600
+F 0 "F1" V 2775 2600 50  0000 C CNN
+F 1 "RXEF050" V 2866 2600 50  0000 C CNN
+F 2 "Capacitor_THT:C_Disc_D8.0mm_W2.5mm_P5.00mm" H 3050 2400 50  0001 L CNN
+F 3 "https://akizukidenshi.com/download/ds/tyco/rxef050.pdf" H 3000 2600 50  0001 C CNN
+	1    3000 2600
+	0    1    1    0
+$EndComp
+Connection ~ 3350 2600
+$Comp
+L power:PWR_FLAG #FLG02
+U 1 1 607F72AB
+P 3300 2600
+F 0 "#FLG02" H 3300 2675 50  0001 C CNN
+F 1 "PWR_FLAG" H 3300 2773 50  0000 C CNN
+F 2 "" H 3300 2600 50  0001 C CNN
+F 3 "~" H 3300 2600 50  0001 C CNN
+	1    3300 2600
+	1    0    0    -1
+$EndComp
+Connection ~ 3300 2600
+Wire Wire Line
+	3300 2600 3350 2600
+Connection ~ 6200 2600
+$Comp
+L Connector:Conn_01x04_Male J4
+U 1 1 60516F4C
+P 10600 9050
+F 0 "J4" H 10708 9331 50  0000 C CNN
+F 1 "Conn_01x04_Male" H 10708 9240 50  0000 C CNN
+F 2 "Connector_PinHeader_2.54mm:PinHeader_1x04_P2.54mm_Horizontal" H 10600 9050 50  0001 C CNN
+F 3 "~" H 10600 9050 50  0001 C CNN
+	1    10600 9050
+	1    0    0    -1
+$EndComp
+Wire Wire Line
+	12150 4600 12150 9050
+Wire Wire Line
+	10800 9050 12150 9050
+Wire Wire Line
+	10800 9150 12250 9150
+$Comp
+L power:GND #PWR021
+U 1 1 60552736
+P 11550 9250
+F 0 "#PWR021" H 11550 9000 50  0001 C CNN
+F 1 "GND" H 11555 9077 50  0000 C CNN
+F 2 "" H 11550 9250 50  0001 C CNN
+F 3 "" H 11550 9250 50  0001 C CNN
+	1    11550 9250
+	1    0    0    -1
+$EndComp
+Wire Wire Line
+	10800 9250 11200 9250
+$Comp
+L Device:CP C21
+U 1 1 6056AB32
+P 11200 9100
+F 0 "C21" H 11085 9054 50  0000 R CNN
+F 1 "10u" H 11085 9145 50  0000 R CNN
+F 2 "Capacitor_THT:C_Axial_L5.1mm_D3.1mm_P7.50mm_Horizontal" H 11238 8950 50  0001 C CNN
+F 3 "~" H 11200 9100 50  0001 C CNN
+	1    11200 9100
+	1    0    0    -1
+$EndComp
+Connection ~ 11200 9250
+Wire Wire Line
+	11200 9250 11550 9250
+$Comp
+L power:VDD #PWR020
+U 1 1 60571ADD
+P 11550 8950
+F 0 "#PWR020" H 11550 8800 50  0001 C CNN
+F 1 "VDD" H 11565 9123 50  0000 C CNN
+F 2 "" H 11550 8950 50  0001 C CNN
+F 3 "" H 11550 8950 50  0001 C CNN
+	1    11550 8950
+	1    0    0    -1
+$EndComp
+Wire Wire Line
+	10800 8950 11200 8950
+Connection ~ 11200 8950
+Wire Wire Line
+	11200 8950 11550 8950
+$Comp
+L Connector:Conn_01x02_Male J1
+U 1 1 6086A811
+P 2100 2600
+F 0 "J1" H 2208 2781 50  0000 C CNN
+F 1 "Conn_01x02_Male" H 2208 2690 50  0000 C CNN
+F 2 "Connector_PinHeader_2.54mm:PinHeader_1x02_P2.54mm_Horizontal" H 2100 2600 50  0001 C CNN
+F 3 "~" H 2100 2600 50  0001 C CNN
+	1    2100 2600
+	1    0    0    -1
+$EndComp
+Wire Wire Line
+	11200 2600 11300 2600
+Connection ~ 11200 2600
+Connection ~ 10700 2600
+Connection ~ 10500 2600
+Wire Wire Line
+	10500 2600 6200 2600
+Wire Wire Line
+	10500 2600 10600 2600
+Connection ~ 11100 2600
+Connection ~ 11000 2600
+Wire Wire Line
+	11100 2600 11200 2600
+Wire Wire Line
+	11000 2600 11100 2600
+Connection ~ 10900 2600
+Connection ~ 10800 2600
+Wire Wire Line
+	10900 2600 11000 2600
+Wire Wire Line
+	10800 2600 10900 2600
+Connection ~ 10600 2600
+Wire Wire Line
+	10700 2600 10800 2600
+Wire Wire Line
+	10600 2600 10700 2600
+Wire Wire Line
+	10800 3800 10800 3100
+Wire Wire Line
+	10700 3700 10700 3100
+Wire Wire Line
+	10600 3250 10600 3100
+Wire Wire Line
+	10500 3300 10500 3100
+Wire Wire Line
+	11300 5000 11300 3100
+Wire Wire Line
+	11200 5100 11200 3100
+Wire Wire Line
+	11100 5200 11100 3100
+Wire Wire Line
+	11000 4000 11000 3100
+Wire Wire Line
+	10900 3100 10900 3900
+$Comp
+L Connector_Generic:Conn_02x09_Odd_Even J5
+U 1 1 604D5366
+P 10900 2900
+F 0 "J5" V 10996 2412 50  0000 R CNN
+F 1 "Conn_02x09_Odd_Even" V 10905 2412 50  0000 R CNN
+F 2 "Connector_PinHeader_2.54mm:PinHeader_2x09_P2.54mm_Horizontal" H 10900 2900 50  0001 C CNN
+F 3 "~" H 10900 2900 50  0001 C CNN
+	1    10900 2900
+	0    1    -1   0
+$EndComp
+$Comp
+L power:VDD #PWR0101
+U 1 1 6045E392
+P 12950 2800
+F 0 "#PWR0101" H 12950 2650 50  0001 C CNN
+F 1 "VDD" H 12965 2973 50  0000 C CNN
+F 2 "" H 12950 2800 50  0001 C CNN
+F 3 "" H 12950 2800 50  0001 C CNN
+	1    12950 2800
+	1    0    0    -1
+$EndComp
+Wire Wire Line
+	12950 2800 13650 2800
+Wire Wire Line
+	13650 2800 13650 2600
+Connection ~ 3200 2900
+Wire Wire Line
+	3200 2700 3200 2900
+Connection ~ 2800 2700
+Wire Wire Line
+	2800 2700 3200 2700
 $Comp
 L power:PWR_FLAG #FLG01
@@
 	1    0    0    1
 $EndComp
-Wire Wire Line
-	11450 4100 10700 4100
-Connection ~ 3200 3550
-$Comp
-L Device:Polyfuse F1
-U 1 1 62039685
-P 3000 2600
-F 0 "F1" V 2775 2600 50  0000 C CNN
-F 1 "RXEF050" V 2866 2600 50  0000 C CNN
-F 2 "Capacitor_THT:C_Disc_D8.0mm_W2.5mm_P5.00mm" H 3050 2400 50  0001 L CNN
-F 3 "https://akizukidenshi.com/download/ds/tyco/rxef050.pdf" H 3000 2600 50  0001 C CNN
-	1    3000 2600
-	0    1    1    0
-$EndComp
-Connection ~ 2800 2700
-Wire Wire Line
-	2800 2700 3200 2700
-Wire Wire Line
-	2600 2700 2800 2700
-Connection ~ 3350 2600
+$Comp
+L Diode:1N4007 D3
+U 1 1 6044A8F3
+P 2700 2600
+F 0 "D3" H 2700 2383 50  0000 C CNN
+F 1 "1N4007" H 2700 2474 50  0000 C CNN
+F 2 "Diode_THT:D_DO-41_SOD81_P2.54mm_Vertical_AnodeUp" H 2700 2425 50  0001 C CNN
+F 3 "http://www.vishay.com/docs/88503/1n4001.pdf" H 2700 2600 50  0001 C CNN
+	1    2700 2600
+	-1   0    0    1
+$EndComp
 Wire Wire Line
 	3150 2600 3300 2600
-$Comp
-L power:PWR_FLAG #FLG02
-U 1 1 607F72AB
-P 3300 2600
-F 0 "#FLG02" H 3300 2675 50  0001 C CNN
-F 1 "PWR_FLAG" H 3300 2773 50  0000 C CNN
-F 2 "" H 3300 2600 50  0001 C CNN
-F 3 "~" H 3300 2600 50  0001 C CNN
-	1    3300 2600
-	1    0    0    -1
-$EndComp
-Connection ~ 3300 2600
-Wire Wire Line
-	3300 2600 3350 2600
-Wire Wire Line
-	2600 2600 2850 2600
-Connection ~ 6200 2600
-$Comp
-L Connector:Conn_01x04_Male J4
-U 1 1 60516F4C
-P 10600 9050
-F 0 "J4" H 10708 9331 50  0000 C CNN
-F 1 "Conn_01x04_Male" H 10708 9240 50  0000 C CNN
-F 2 "Connector_PinHeader_2.54mm:PinHeader_1x04_P2.54mm_Horizontal" H 10600 9050 50  0001 C CNN
-F 3 "~" H 10600 9050 50  0001 C CNN
-	1    10600 9050
-	1    0    0    -1
-$EndComp
-Wire Wire Line
-	12150 4600 12150 9050
-Wire Wire Line
-	10800 9050 12150 9050
-Wire Wire Line
-	10800 9150 12250 9150
-$Comp
-L power:GND #PWR021
-U 1 1 60552736
-P 11550 9250
-F 0 "#PWR021" H 11550 9000 50  0001 C CNN
-F 1 "GND" H 11555 9077 50  0000 C CNN
-F 2 "" H 11550 9250 50  0001 C CNN
-F 3 "" H 11550 9250 50  0001 C CNN
-	1    11550 9250
-	1    0    0    -1
-$EndComp
-Wire Wire Line
-	10800 9250 11200 9250
-$Comp
-L Device:CP C21
-U 1 1 6056AB32
-P 11200 9100
-F 0 "C21" H 11085 9054 50  0000 R CNN
-F 1 "10u" H 11085 9145 50  0000 R CNN
-F 2 "Capacitor_THT:C_Axial_L5.1mm_D3.1mm_P7.50mm_Horizontal" H 11238 8950 50  0001 C CNN
-F 3 "~" H 11200 9100 50  0001 C CNN
-	1    11200 9100
-	1    0    0    -1
-$EndComp
-Connection ~ 11200 9250
-Wire Wire Line
-	11200 9250 11550 9250
-$Comp
-L power:VDD #PWR020
-U 1 1 60571ADD
-P 11550 8950
-F 0 "#PWR020" H 11550 8800 50  0001 C CNN
-F 1 "VDD" H 11565 9123 50  0000 C CNN
-F 2 "" H 11550 8950 50  0001 C CNN
-F 3 "" H 11550 8950 50  0001 C CNN
-	1    11550 8950
-	1    0    0    -1
-$EndComp
-Wire Wire Line
-	10800 8950 11200 8950
-Connection ~ 11200 8950
-Wire Wire Line
-	11200 8950 11550 8950
-$Comp
-L Connector:Conn_01x02_Male J1
-U 1 1 6086A811
-P 2400 2600
-F 0 "J1" H 2508 2781 50  0000 C CNN
-F 1 "Conn_01x02_Male" H 2508 2690 50  0000 C CNN
-F 2 "Connector_PinHeader_2.54mm:PinHeader_1x02_P2.54mm_Horizontal" H 2400 2600 50  0001 C CNN
-F 3 "~" H 2400 2600 50  0001 C CNN
-	1    2400 2600
-	1    0    0    -1
-$EndComp
-Wire Wire Line
-	11200 2600 11300 2600
-Connection ~ 11200 2600
-Connection ~ 10700 2600
-Connection ~ 10500 2600
-Wire Wire Line
-	10500 2600 6200 2600
-Wire Wire Line
-	10500 2600 10600 2600
-Connection ~ 11100 2600
-Connection ~ 11000 2600
-Wire Wire Line
-	11100 2600 11200 2600
-Wire Wire Line
-	11000 2600 11100 2600
-Connection ~ 10900 2600
-Connection ~ 10800 2600
-Wire Wire Line
-	10900 2600 11000 2600
-Wire Wire Line
-	10800 2600 10900 2600
-Connection ~ 10600 2600
-Wire Wire Line
-	10700 2600 10800 2600
-Wire Wire Line
-	10600 2600 10700 2600
-Wire Wire Line
-	10800 3800 10800 3100
-Wire Wire Line
-	10700 3700 10700 3100
-Wire Wire Line
-	10600 3250 10600 3100
-Wire Wire Line
-	10500 3300 10500 3100
-Wire Wire Line
-	11300 5000 11300 3100
-Wire Wire Line
-	11200 5100 11200 3100
-Wire Wire Line
-	11100 5200 11100 3100
-Wire Wire Line
-	11000 4000 11000 3100
-Wire Wire Line
-	10900 3100 10900 3900
-$Comp
-L Connector_Generic:Conn_02x09_Odd_Even J5
-U 1 1 604D5366
-P 10900 2900
-F 0 "J5" V 10996 2412 50  0000 R CNN
-F 1 "Conn_02x09_Odd_Even" V 10905 2412 50  0000 R CNN
-F 2 "Connector_PinHeader_2.54mm:PinHeader_2x09_P2.54mm_Horizontal" H 10900 2900 50  0001 C CNN
-F 3 "~" H 10900 2900 50  0001 C CNN
-	1    10900 2900
-	0    1    -1   0
-$EndComp
+Wire Wire Line
+	2300 2600 2550 2600
+Wire Wire Line
+	2300 2700 2800 2700
 $EndSCHEMATC

Commit message: 20210604
Parts:
- removed C4: 10u, Capacitor_THT:CP_Radial_D5.0mm_P2.50mm, symbol Device:CP
- removed C5: 0.1u, Capacitor_THT:C_Disc_D3.0mm_W1.6mm_P2.50mm, symbol Device:C
- removed D1: LED, LED_THT:LED_D3.0mm, symbol Device:LED
- removed R1: 1k, Resistor_THT:R_Axial_DIN0204_L3.6mm_D1.6mm_P7.62mm_Horizontal, symbol Device:R
Connections:
- net GND: now also D3.2 (A)
- net VDD: now also C8.2, C9.1, J5.10 (Pin_10), J5.12 (Pin_12), J5.14 (Pin_14), J5.16 (Pin_16), J5.18 (Pin_18), J5.2 (Pin_2), J5.4 (Pin_4), J5.6 (Pin_6), J5.8 (Pin_8)
- net at D3.1 (K): now also C2.1, C3.1, F1.1, U2.1 (IN), U3.1 (IN); no longer F1.2
- net at J1.1 (Pin_1): now also F1.2; no longer D3.2 (A)
Other:
- moved on the sheet: D3, F1
Changed lines of the file:
@@
 	1    0    0    -1
 $EndComp
-$Comp
-L Device:R R1
-U 1 1 60A9C419
-P 4500 2600
-F 0 "R1" V 4700 2600 50  0000 C CNN
-F 1 "1k" V 4600 2600 50  0000 C CNN
-F 2 "Resistor_THT:R_Axial_DIN0204_L3.6mm_D1.6mm_P7.62mm_Horizontal" V 4430 2600 50  0001 C CNN
-F 3 "~" H 4500 2600 50  0001 C CNN
-	1    4500 2600
-	0    -1   -1   0
-$EndComp
-Wire Wire Line
-	4300 2600 4350 2600
 Connection ~ 4300 2600
-$Comp
-L Device:LED D1
-U 1 1 60B0C789
-P 5350 2750
-F 0 "D1" H 5343 2495 50  0000 C CNN
-F 1 "LED" H 5343 2586 50  0000 C CNN
-F 2 "LED_THT:LED_D3.0mm" H 5350 2750 50  0001 C CNN
-F 3 "~" H 5350 2750 50  0001 C CNN
-	1    5350 2750
-	0    -1   -1   0
-$EndComp
-Wire Wire Line
-	3900 2900 4800 2900
-Wire Wire Line
-	4650 2600 4800 2600
-Connection ~ 4800 2600
 $Comp
 L Device:CP C9
@@
 	1    6200 2750
 	1    0    0    -1
-$EndComp
-$Comp
-L Device:CP C4
-U 1 1 60B5E5AB
-P 4800 2750
-F 0 "C4" H 4685 2704 50  0000 R CNN
-F 1 "10u" H 4685 2795 50  0000 R CNN
-F 2 "Capacitor_THT:CP_Radial_D5.0mm_P2.50mm" H 4838 2600 50  0001 C CNN
-F 3 "~" H 4800 2750 50  0001 C CNN
-	1    4800 2750
-	1    0    0    -1
-$EndComp
-Connection ~ 5100 2600
-Wire Wire Line
-	5100 2600 5350 2600
-Wire Wire Line
-	4800 2600 5100 2600
-Connection ~ 5350 2600
-$Comp
-L Device:C C5
-U 1 1 60B80873
-P 5100 2750
-F 0 "C5" H 4985 2704 50  0000 R CNN
-F 1 "0.1u" H 4985 2795 50  0000 R CNN
-F 2 "Capacitor_THT:C_Disc_D3.0mm_W1.6mm_P2.50mm" H 5138 2600 50  0001 C CNN
-F 3 "~" H 5100 2750 50  0001 C CNN
-	1    5100 2750
-	-1   0    0    1
 $EndComp
 $Comp
@@
 	-1   0    0    1
 $EndComp
-Wire Wire Line
-	5350 2600 5700 2600
 Connection ~ 5700 2600
 Wire Wire Line
 	5700 2600 6200 2600
-Wire Wire Line
-	4800 2900 5100 2900
-Connection ~ 4800 2900
-Connection ~ 5100 2900
-Wire Wire Line
-	5100 2900 5350 2900
-Connection ~ 5350 2900
-Wire Wire Line
-	5350 2900 5700 2900
 Connection ~ 5700 2900
 Wire Wire Line
@@
 L Device:Polyfuse F1
 U 1 1 62039685
-P 3000 2600
-F 0 "F1" V 2775 2600 50  0000 C CNN
-F 1 "RXEF050" V 2866 2600 50  0000 C CNN
-F 2 "Capacitor_THT:C_Disc_D8.0mm_W2.5mm_P5.00mm" H 3050 2400 50  0001 L CNN
-F 3 "https://akizukidenshi.com/download/ds/tyco/rxef050.pdf" H 3000 2600 50  0001 C CNN
-	1    3000 2600
+P 2700 2600
+F 0 "F1" V 2475 2600 50  0000 C CNN
+F 1 "RXEF050" V 2566 2600 50  0000 C CNN
+F 2 "Capacitor_THT:C_Disc_D8.0mm_W2.5mm_P5.00mm" H 2750 2400 50  0001 L CNN
+F 3 "https://akizukidenshi.com/download/ds/tyco/rxef050.pdf" H 2700 2600 50  0001 C CNN
+	1    2700 2600
 	0    1    1    0
 $EndComp
@@
 Connection ~ 2800 2700
 Wire Wire Line
-	2800 2700 3200 2700
+	2800 2700 2850 2700
 $Comp
 L power:PWR_FLAG #FLG01
@@
 L Diode:1N4007 D3
 U 1 1 6044A8F3
-P 2700 2600
-F 0 "D3" H 2700 2383 50  0000 C CNN
-F 1 "1N4007" H 2700 2474 50  0000 C CNN
-F 2 "Diode_THT:D_DO-41_SOD81_P2.54mm_Vertical_AnodeUp" H 2700 2425 50  0001 C CNN
-F 3 "http://www.vishay.com/docs/88503/1n4001.pdf" H 2700 2600 50  0001 C CNN
-	1    2700 2600
+P 3000 2650
+F 0 "D3" H 3000 2433 50  0000 C CNN
+F 1 "1N4007" H 3000 2524 50  0000 C CNN
+F 2 "Diode_THT:D_DO-41_SOD81_P2.54mm_Vertical_AnodeUp" H 3000 2475 50  0001 C CNN
+F 3 "http://www.vishay.com/docs/88503/1n4001.pdf" H 3000 2650 50  0001 C CNN
+	1    3000 2650
 	-1   0    0    1
 $EndComp
 Wire Wire Line
+	2300 2600 2550 2600
+Wire Wire Line
+	2300 2700 2800 2700
+Wire Wire Line
+	3900 2900 5700 2900
+Wire Wire Line
+	4300 2600 5700 2600
+Wire Wire Line
+	2850 2600 3150 2600
+Wire Wire Line
+	3150 2650 3150 2600
+Connection ~ 3150 2600
+Wire Wire Line
 	3150 2600 3300 2600
 Wire Wire Line
-	2300 2600 2550 2600
-Wire Wire Line
-	2300 2700 2800 2700
+	2850 2650 2850 2700
+Connection ~ 2850 2700
+Wire Wire Line
+	2850 2700 3200 2700
 $EndSCHEMATC

Commit message: メイン飛んだ
Parts:
- added C24: 10u, Capacitor_THT:CP_Radial_D5.0mm_P2.50mm, symbol Device:CP
- added C25: 0.1u, Capacitor_THT:C_Disc_D3.0mm_W1.6mm_P2.50mm, symbol Device:C
- added D3: LED, LED_THT:LED_D5.0mm, symbol Device:LED
- added R40: 1k, Resistor_THT:R_Axial_DIN0204_L3.6mm_D1.6mm_P7.62mm_Horizontal, symbol Device:R
- renumbered C12 to C10, C14 to C11, C15 to C12, C16 to C13, C17 to C14, C18 to C15, C19 to C16, C20 to C17, C21 to C18, C22 to C19, C6 to C4, C7 to C5, C8 to C6, C9 to C7, C10 to C8, C11 to C9, D3 to D1, R2 to R1, R11 to R10, R12 to R11, R13 to R12, R14 to R13, R15 to R14, R16 to R15, R17 to R16, R18 to R17, R19 to R18, R20 to R19, R3 to R2, R21 to R20, R22 to R21, R23 to R22, R4 to R3, R5 to R4, R6 to R5, R7 to R6, R8 to R7, R9 to R8, R10 to R9
Connections:
- net GND: now also C24.2, C25.1, D3.1 (K)
- net VDD: now also R40.1; no longer C6.2, C7.1, J5.10 (Pin_10), J5.12 (Pin_12), J5.14 (Pin_14), J5.16 (Pin_16), J5.18 (Pin_18), J5.2 (Pin_2), J5.4 (Pin_4), J5.6 (Pin_6), J5.8 (Pin_8)
- net Sheet60E5A5FF/B: now reaches J2.3 (Pin_3), U4.10 (OSC2/CLKO/RPA3/PMA0/RA3), U5.10 (B)
- net Sheet60E5A5FF/C: now reaches J2.4 (Pin_4), U4.11 (SOSCI/RPB4/RB4), U5.9 (C)
- net Sheet60D32BD3/SCL: now reaches J4.3 (Pin_3), U4.17 (TCK/RPB8/SCL1/CTED10/PMD4/RB8)
- net Sheet60D32BD3/SDA: now reaches J4.2 (Pin_2), U4.18 (TDO/RPB9/SDA1/CTED4/PMD3/RB9)
- net Sheet60E5A5FF/A+: now reaches J5.3 (Pin_3), U4.25 (CVREFOUT/AN10/C3INB/RPB14/SCK1/CTED5/PMWR/RB14)
- net Sheet60E5A5FF/A: now reaches J2.2 (Pin_2), U4.9 (OSC1/CLKI/RPA2/RA2), U5.11 (A)
- new net Sheet60E5A5FF/A-: C24.1, C25.2, C6.2, C7.1, D3.2 (A), J5.10 (Pin_10), J5.12 (Pin_12), J5.14 (Pin_14), J5.16 (Pin_16), J5.18 (Pin_18), J5.2 (Pin_2), J5.4 (Pin_4), J5.6 (Pin_6), J5.8 (Pin_8), R40.2
