File: Circuit/Mother/file60E5A5FF.sch (KiCad schematic (older format))
At the start: 17 parts, among them J2 Conn_02x08_Odd_Even, U1 4051

Commit message: メイン飛んだ
Parts:
- renumbered C2 to C23, J2 to J11, R1 to R26, R2 to R27, R3 to R28, R4 to R29, R5 to R30, R6 to R31, R9 to R32, R10 to R33, R11 to R34, R12 to R35, R13 to R36, R14 to R37, R15 to R38, R16 to R39, U1 to U10
Connections:
- net A-: now also J11.1 (Pin_1), J11.2 (Pin_2), R39.2
- net VDD: no longer J11.2 (Pin_2)
Changed lines of the file:
@@
 $EndDescr
 $Comp
-L 4xxx:4051 U1
+L 4xxx:4051 U10
 U 1 1 60481B08
 P 5350 2950
-F 0 "U1" H 5894 2996 50  0000 L CNN
+F 0 "U10" H 5894 2996 50  0000 L CNN
 F 1 "4051" H 5894 2905 50  0000 L CNN
 F 2 "Package_DIP:DIP-16_W7.62mm" H 5350 2950 50  0001 C CNN
@@
 	5350 3850 5450 3850
 $Comp
-L power:GND #PWR03
+L power:GND #PWR043
 U 1 1 60482D4F
 P 4250 3850
-F 0 "#PWR03" H 4250 3600 50  0001 C CNN
+F 0 "#PWR043" H 4250 3600 50  0001 C CNN
 F 1 "GND" H 4255 3677 50  0000 C CNN
 F 2 "" H 4250 3850 50  0001 C CNN
@@
 $EndComp
 $Comp
-L Device:C C2
+L Device:C C23
 U 1 1 604831DD
 P 5200 1950
-F 0 "C2" V 4948 1950 50  0000 C CNN
+F 0 "C23" V 4948 1950 50  0000 C CNN
 F 1 "0.1u" V 5039 1950 50  0000 C CNN
 F 2 "Capacitor_THT:C_Disc_D3.0mm_W1.6mm_P2.50mm" H 5238 1800 50  0001 C CNN
@@
 	5350 1950 5350 2050
 $Comp
-L power:GND #PWR04
+L power:GND #PWR044
 U 1 1 6048C611
 P 5050 1950
-F 0 "#PWR04" H 5050 1700 50  0001 C CNN
+F 0 "#PWR044" H 5050 1700 50  0001 C CNN
 F 1 "GND" H 5055 1777 50  0000 C CNN
 F 2 "" H 5050 1950 50  0001 C CNN
@@
 $EndComp
 $Comp
-L Device:R R1
+L Device:R R26
 U 1 1 604A613D
 P 3450 2400
-F 0 "R1" V 3450 2400 50  0000 C CNN
+F 0 "R26" V 3450 2400 50  0000 C CNN
 F 1 "1Meg" V 3400 2600 50  0000 C CNN
 F 2 "Resistor_THT:R_Axial_DIN0204_L3.6mm_D1.6mm_P7.62mm_Horizontal" V 3380 2400 50  0001 C CNN
@@
 $EndComp
 $Comp
-L Device:R R2
+L Device:R R27
 U 1 1 604AAB33
 P 3450 2500
-F 0 "R2" V 3450 2500 50  0000 C CNN
+F 0 "R27" V 3450 2500 50  0000 C CNN
 F 1 "1Meg" V 3400 2700 50  0000 C CNN
 F 2 "Resistor_THT:R_Axial_DIN0204_L3.6mm_D1.6mm_P7.62mm_Horizontal" V 3380 2500 50  0001 C CNN
@@
 $EndComp
 $Comp
-L Device:R R3
+L Device:R R28
 U 1 1 604AAE48
 P 3450 2600
-F 0 "R3" V 3450 2600 50  0000 C CNN
+F 0 "R28" V 3450 2600 50  0000 C CNN
 F 1 "1Meg" V 3400 2800 50  0000 C CNN
 F 2 "Resistor_THT:R_Axial_DIN0204_L3.6mm_D1.6mm_P7.62mm_Horizontal" V 3380 2600 50  0001 C CNN
@@
 $EndComp
 $Comp
-L Device:R R4
+L Device:R R29
 U 1 1 604AB14B
 P 3450 2700
-F 0 "R4" V 3450 2700 50  0000 C CNN
+F 0 "R29" V 3450 2700 50  0000 C CNN
 F 1 "1Meg" V 3400 2900 50  0000 C CNN
 F 2 "Resistor_THT:R_Axial_DIN0204_L3.6mm_D1.6mm_P7.62mm_Horizontal" V 3380 2700 50  0001 C CNN
@@
 $EndComp
 $Comp
-L Device:R R5
+L Device:R R30
 U 1 1 604AB466
 P 3450 2800
-F 0 "R5" V 3450 2800 50  0000 C CNN
+F 0 "R30" V 3450 2800 50  0000 C CNN
 F 1 "1Meg" V 3400 3000 50  0000 C CNN
 F 2 "Resistor_THT:R_Axial_DIN0204_L3.6mm_D1.6mm_P7.62mm_Horizontal" V 3380 2800 50  0001 C CNN
@@
 $EndComp
 $Comp
-L Device:R R6
+L Device:R R31
 U 1 1 604AB730
 P 3450 2900
-F 0 "R6" V 3450 2900 50  0000 C CNN
+F 0 "R31" V 3450 2900 50  0000 C CNN
 F 1 "1Meg" V 3400 3100 50  0000 C CNN
 F 2 "Resistor_THT:R_Axial_DIN0204_L3.6mm_D1.6mm_P7.62mm_Horizontal" V 3380 2900 50  0001 C CNN
@@
 Connection ~ 3300 2150
 $Comp
-L power:VDD #PWR05
+L power:VDD #PWR045
 U 1 1 604CE1F8
 P 5350 1950
-F 0 "#PWR05" H 5350 1800 50  0001 C CNN
+F 0 "#PWR045" H 5350 1800 50  0001 C CNN
 F 1 "VDD" H 5365 2123 50  0000 C CNN
 F 2 "" H 5350 1950 50  0001 C CNN
@@
 	4250 3250 4250 3850
 $Comp
-L Connector_Generic:Conn_02x08_Odd_Even J2
+L Connector_Generic:Conn_02x08_Odd_Even J11
 U 1 1 602DFCF7
 P 4150 2750
-F 0 "J2" H 4200 2125 50  0000 C CNN
+F 0 "J11" H 4200 2125 50  0000 C CNN
 F 1 "Conn_02x08_Odd_Even" H 4200 2216 50  0000 C CNN
 F 2 "Connector_PinHeader_2.54mm:PinHeader_2x08_P2.54mm_Horizontal" H 4150 2750 50  0001 C CNN
@@
 	3300 1500 5850 1500
 $Comp
-L Device:R R9
+L Device:R R32
 U 1 1 6041C195
 P 4600 2350
-F 0 "R9" V 4600 2350 50  0000 C CNN
+F 0 "R32" V 4600 2350 50  0000 C CNN
 F 1 "220" V 4550 2550 50  0000 C CNN
 F 2 "Resistor_THT:R_Axial_DIN0204_L3.6mm_D1.6mm_P7.62mm_Horizontal" V 4530 2350 50  0001 C CNN
@@
 	4750 2350 4850 2350
 $Comp
-L Device:R R10
+L Device:R R33
 U 1 1 60427657
 P 4600 2450
-F 0 "R10" V 4600 2450 50  0000 C CNN
+F 0 "R33" V 4600 2450 50  0000 C CNN
 F 1 "220" V 4550 2650 50  0000 C CNN
 F 2 "Resistor_THT:R_Axial_DIN0204_L3.6mm_D1.6mm_P7.62mm_Horizontal" V 4530 2450 50  0001 C CNN
@@
 $EndComp
 $Comp
-L Device:R R11
+L Device:R R34
 U 1 1 60427859
 P 4600 2550
-F 0 "R11" V 4600 2550 50  0000 C CNN
+F 0 "R34" V 4600 2550 50  0000 C CNN
 F 1 "220" V 4550 2750 50  0000 C CNN
 F 2 "Resistor_THT:R_Axial_DIN0204_L3.6mm_D1.6mm_P7.62mm_Horizontal" V 4530 2550 50  0001 C CNN
@@
 $EndComp
 $Comp
-L Device:R R12
+L Device:R R35
 U 1 1 60427A23
 P 4600 2650
-F 0 "R12" V 4600 2650 50  0000 C CNN
+F 0 "R35" V 4600 2650 50  0000 C CNN
 F 1 "220" V 4550 2850 50  0000 C CNN
 F 2 "Resistor_THT:R_Axial_DIN0204_L3.6mm_D1.6mm_P7.62mm_Horizontal" V 4530 2650 50  0001 C CNN
@@
 $EndComp
 $Comp
-L Device:R R13
+L Device:R R36
 U 1 1 60427BF9
 P 4600 2750
-F 0 "R13" V 4600 2750 50  0000 C CNN
+F 0 "R36" V 4600 2750 50  0000 C CNN
 F 1 "220" V 4550 2950 50  0000 C CNN
 F 2 "Resistor_THT:R_Axial_DIN0204_L3.6mm_D1.6mm_P7.62mm_Horizontal" V 4530 2750 50  0001 C CNN
@@
 $EndComp
 $Comp
-L Device:R R14
+L Device:R R37
 U 1 1 60427DEB
 P 4600 2850
-F 0 "R14" V 4600 2850 50  0000 C CNN
+F 0 "R37" V 4600 2850 50  0000 C CNN
 F 1 "220" V 4550 3050 50  0000 C CNN
 F 2 "Resistor_THT:R_Axial_DIN0204_L3.6mm_D1.6mm_P7.62mm_Horizontal" V 4530 2850 50  0001 C CNN
@@
 $EndComp
 $Comp
-L Device:R R15
+L Device:R R38
 U 1 1 60427FD9
 P 4600 2950
-F 0 "R15" V 4600 2950 50  0000 C CNN
+F 0 "R38" V 4600 2950 50  0000 C CNN
 F 1 "220" V 4550 3150 50  0000 C CNN
 F 2 "Resistor_THT:R_Axial_DIN0204_L3.6mm_D1.6mm_P7.62mm_Horizontal" V 4530 2950 50  0001 C CNN
@@
 $EndComp
 $Comp
-L Device:R R16
+L Device:R R39
 U 1 1 604281E3
 P 4600 3050
-F 0 "R16" V 4600 3050 50  0000 C CNN
+F 0 "R39" V 4600 3050 50  0000 C CNN
 F 1 "220" V 4550 3250 50  0000 C CNN
 F 2 "Resistor_THT:R_Axial_DIN0204_L3.6mm_D1.6mm_P7.62mm_Horizontal" V 4530 3050 50  0001 C CNN
@@
 Wire Wire Line
 	4350 3000 3300 3000
-$Comp
-L power:VDD #PWR?
-U 1 1 60416052
-P 3150 3050
-F 0 "#PWR?" H 3150 2900 50  0001 C CNN
-F 1 "VDD" H 3165 3223 50  0000 C CNN
-F 2 "" H 3150 3050 50  0001 C CNN
-F 3 "" H 3150 3050 50  0001 C CNN
-	1    3150 3050
-	1    0    0    -1
-$EndComp
-Wire Wire Line
-	3850 3050 3150 3050
 Text HLabel 5850 2250 2    50   Output ~ 0
 A-
@@
 Text HLabel 1900 3550 0    50   Input ~ 0
 C
+Wire Wire Line
+	3850 2950 3850 3050
+Connection ~ 3850 2950
+Wire Wire Line
+	3300 3000 3300 3100
+Wire Wire Line
+	3300 3100 4350 3100
+Wire Wire Line
+	4350 3100 4350 3050
+Connection ~ 3300 3000
+Connection ~ 4350 3050
 $EndSCHEMATC
