File: Circuit/peripheral/peripheral.sch (KiCad schematic (older format))
At the start: 120 parts

Commit message: 回路完成
Parts:
- added SW9: SW_DIP_x01, symbol Switch:SW_DIP_x01
- gave numbers to parts that had none: 120
Connections:
- net at J24.1 (Pin_1): now also SW9.1; no longer J28.1
- new net: J28.1, SW9.2
- no-connect marks 38 -> 43
Other:
- moved on the sheet: J28
