File: Circuit/Mother2/Mother.sch (KiCad schematic (older format))
At the start: 57 parts, among them J1 Conn_01x02_Male, J2 Conn_01x05_Male, J3 Conn_02x09_Odd_Even, J4 Conn_01x04_Male, J5 Conn_02x09_Odd_Even, J6 Conn_PIC_ICSP_ICD, J7 Conn_01x05_Male, U1 74HC00, U2 BP5293-33, U3 BP5293-50, U4 PIC32MX110F016B-I_SP, U5 4051, U6 TLP785

Commit message: 20210604
Parts:
- renumbered C12 to C10, C14 to C11, C15 to C12, C16 to C13, C17 to C14, C18 to C15, C19 to C16, C20 to C17, C21 to C18, C22 to C19, C6 to C4, C7 to C5, C8 to C6, C9 to C7, C10 to C8, C11 to C9, D3 to D1, R2 to R1, R11 to R10, R12 to R11, R13 to R12, R14 to R13, R15 to R14, R16 to R15, R17 to R16, R18 to R17, R19 to R18, R20 to R19, R3 to R2, R21 to R20, R22 to R21, R23 to R22, R4 to R3, R5 to R4, R6 to R5, R7 to R6, R8 to R7, R9 to R8, R10 to R9
Connections:
- net GND: now also D1.2 (A)
- net Sheet60E5A5FF/B: now reaches J2.3 (Pin_3), U4.10 (OSC2/CLKO/RPA3/PMA0/RA3), U5.10 (B)
- net Sheet60E5A5FF/C: now reaches J2.4 (Pin_4), U4.11 (SOSCI/RPB4/RB4), U5.9 (C)
- net Sheet60D32BD3/SCL: now reaches J4.3 (Pin_3), U4.17 (TCK/RPB8/SCL1/CTED10/PMD4/RB8)
- net Sheet60D32BD3/SDA: now reaches J4.2 (Pin_2), U4.18 (TDO/RPB9/SDA1/CTED4/PMD3/RB9)
- net Sheet60E5A5FF/A+: now reaches J5.3 (Pin_3), U4.25 (CVREFOUT/AN10/C3INB/RPB14/SCK1/CTED5/PMWR/RB14)
- net Sheet60E5A5FF/A: now reaches J2.2 (Pin_2), U4.9 (OSC1/CLKI/RPA2/RA2), U5.11 (A)
- net at D1.1 (K): now also C2.1, C3.1, F1.1, U2.1 (IN), U3.1 (IN); no longer F1.2
- net at J1.1 (Pin_1): now also F1.2; no longer D1.2 (A)
Other:
- moved on the sheet: D1, F1
