File: Circuit/Display/Display.kicad_pcb (KiCad board)
At the start: 2 copper layers, 29 parts, among them J1 Conn_PIC_ICSP_ICD, J2 Conn_01x04_Female, U1 TBD62783A, U2 PIC16F18854-SO, U3 ULN2803A

Commit message: display
Parts:
- moved BAR1 27.9 mm to (139.7, 71.1)
- moved AFF5 12.7 mm to (124.5, 86.4)
- moved AFF4 12.7 mm to (111.8, 86.4)
Connections:
- AFF1 pad 8: /LED_D0 -> Net-(AFF1-Pad8)
- AFF2 pad 8: /LED_D3 -> Net-(AFF2-Pad8)
- AFF3 pad 8: /LED_D1 -> Net-(AFF3-Pad8)
- AFF4 pad 3: /LED_D4 -> Net-(AFF4-Pad3)
- AFF5 pad 3: /LED_D2 -> Net-(AFF5-Pad3)
Routing:
- net /LED_S6: track 5.08 -> 183.1 mm, vias 0 -> 8
- net /LED_S1: track 15.2 -> 188.0 mm, vias 0 -> 9
- net /LED_S5: track 8.67 -> 175.4 mm, vias 0 -> 8
- net /LED_S0: track 12.7 -> 167.6 mm, vias 0 -> 9
- net /LED_S4: track 25.4 -> 178.9 mm, vias 0 -> 9
- net /LED_S2: track 0.00 -> 147.3 mm, vias 0 -> 6
- net /LED_S3: track 38.1 -> 183.9 mm, vias 0 -> 8
- net /LED_D6: track 35.6 -> 135.9 mm, vias 0 -> 1
- net /LED_D4: track 0.00 -> 86.9 mm
- net /LED_D3: track 0.00 -> 62.8 mm
- net /LED_D0: track 0.00 -> 61.9 mm
- net /LED_D2: track 0.00 -> 51.7 mm
- net /LED_D1: track 0.00 -> 51.5 mm
- net /LED_D5: track 15.2 -> 54.8 mm
- net Net-(R7-Pad2): track 20.3 -> 22.9 mm
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Other:
- copper layers 2 -> 4

Commit message: 20200223
Parts:
- moved R10 36.4 mm to (99.1, 139.7), turned to 0 degrees
- moved C4 31.8 mm to (94.0, 132.1)
- moved J2 30.9 mm to (99.1, 137.2), turned to 180 degrees
- moved R9 21.7 mm to (111.8, 137.2), turned to 0 degrees
- moved D1 17.8 mm to (96.5, 40.6)
- moved D4 10.2 mm to (114.3, 40.6)
- moved D2 5.08 mm to (149.9, 40.6)
- moved D3 2.54 mm to (132.1, 40.6)
Routing:
- net Net-(J2-Pad2): track 13.8 -> 40.6 mm, vias 0 -> 2
- net Net-(J2-Pad3): track 7.62 -> 30.5 mm
- net /LED_D6: track 135.9 -> 153.7 mm
- net /LED_S3: track 183.9 -> 171.2 mm
- net VDD: track 116.2 -> 125.8 mm, vias 4 -> 3
- net /LED_S4: track 178.9 -> 173.8 mm
- net GND: track 144.6 -> 148.2 mm
- net /LED_S5: track 175.4 -> 178.0 mm
- net /LED_S6: track 183.1 -> 184.1 mm

Commit message: mother回路図作成
Parts:
- J1: footprint Connector_PinHeader_2.54mm:PinHeader_1x06_P2.54mm_Vertical -> Connector_PinHeader_2.54mm:PinHeader_1x06_P2.54mm_Horizontal
- J2: footprint Connector_PinSocket_2.54mm:PinSocket_1x04_P2.54mm_Vertical -> Connector_PinHeader_2.54mm:PinHeader_1x04_P2.54mm_Horizontal
- R1, R2, R3, R4, R5, R6, R7: value 4.7k -> 220
- moved C4 6.35 mm to (99.1, 135.9), turned to 90 degrees
- moved J2 5.08 mm to (94.0, 137.2)
Connections:
- AFF1 pad 5: Net-(AFF1-Pad5) -> (no net)
- AFF1 pad 8: Net-(AFF1-Pad8) -> (no net)
- AFF2 pad 5: Net-(AFF2-Pad5) -> (no net)
- AFF2 pad 8: Net-(AFF2-Pad8) -> (no net)
- AFF3 pad 5: Net-(AFF3-Pad5) -> (no net)
- AFF3 pad 8: Net-(AFF3-Pad8) -> (no net)
- AFF4 pad 3: Net-(AFF4-Pad3) -> (no net)
- AFF4 pad 5: Net-(AFF4-Pad5) -> (no net)
- AFF5 pad 3: Net-(AFF5-Pad3) -> (no net)
- AFF5 pad 5: Net-(AFF5-Pad5) -> (no net)
- C4 pad 1: GND -> VDD
- C4 pad 2: VDD -> GND
- J1 pad 6: Net-(J1-Pad6) -> (no net)
- U1 pad 18: Net-(U1-Pad18) -> (no net)
- U3 pad 10: Net-(U3-Pad10) -> (no net)
- U3 pad 11: Net-(U3-Pad11) -> (no net)
Routing:
- net Net-(J2-Pad3): track 30.5 -> 35.6 mm
- net Net-(J2-Pad2): track 40.6 -> 45.7 mm
- net GND: track 148.2 -> 150.9 mm, vias 2 -> 3
- net VDD: track 125.8 -> 126.0 mm, vias 3 -> 4

Commit message: 基板完成
Other:
- board text added: "25x40"

Commit message: 回路完成
Parts:
- J2: value Conn_01x04_Female -> Conn_01x04_Male
- moved C1 45.3 mm to (144.8, 137.2), turned to 0 degrees
- moved U1 25.4 mm to (139.7, 109.2), turned to 0 degrees
- moved U3 25.4 mm to (119.4, 124.5), turned to 180 degrees
- moved BAR1 24.5 mm to (148.6, 94.0), turned to 180 degrees
- moved D1 2.54 mm to (96.5, 43.2), turned to 90 degrees
- moved D2 2.54 mm to (149.9, 43.2), turned to 90 degrees
- moved D3 2.54 mm to (132.1, 43.2), turned to 90 degrees
- moved D4 2.54 mm to (114.3, 43.2), turned to 90 degrees
Connections:
- net Net-(J2-Pad2) renamed /SDA
- net Net-(J2-Pad3) renamed /SCL
- BAR1 pad 1: /LED_S0 -> /LED_D6
- BAR1 pad 10: /LED_S2 -> /LED_D5
- BAR1 pad 11: /LED_D6 -> /LED_S0
- BAR1 pad 12: /LED_D6 -> /LED_S1
- BAR1 pad 13: /LED_D6 -> /LED_S2
- BAR1 pad 14: /LED_D5 -> /LED_S3
- BAR1 pad 15: /LED_D5 -> /LED_S4
- BAR1 pad 16: /LED_D5 -> /LED_S5
- BAR1 pad 17: /LED_D5 -> /LED_S6
- BAR1 pad 18: /LED_D5 -> /LED_S0
- BAR1 pad 19: /LED_D5 -> /LED_S1
- BAR1 pad 2: /LED_S1 -> /LED_D6
- BAR1 pad 20: /LED_D5 -> /LED_S2
- BAR1 pad 3: /LED_S2 -> /LED_D6
- BAR1 pad 4: /LED_S3 -> /LED_D5
- BAR1 pad 5: /LED_S4 -> /LED_D5
- BAR1 pad 6: /LED_S5 -> /LED_D5
- BAR1 pad 7: /LED_S6 -> /LED_D5
- BAR1 pad 8: /LED_S0 -> /LED_D5
- BAR1 pad 9: /LED_S1 -> /LED_D5
- D1 pad 1: /LED_D6 -> /LED_S3
- D1 pad 2: /LED_S3 -> /LED_D6
- D2 pad 1: /LED_D6 -> /LED_S4
- D2 pad 2: /LED_S4 -> /LED_D6
- D3 pad 1: /LED_D6 -> /LED_S5
- D3 pad 2: /LED_S5 -> /LED_D6
- D4 pad 1: /LED_D6 -> /LED_S6
- D4 pad 2: /LED_S6 -> /LED_D6
- U1 pad 11: Net-(R1-Pad2) -> (no net)
- U1 pad 12: Net-(R2-Pad2) -> /LED_D6
- U1 pad 13: Net-(R3-Pad2) -> /LED_D5
- U1 pad 14: Net-(R4-Pad2) -> /LED_D4
- U1 pad 15: Net-(R5-Pad2) -> /LED_D3
- U1 pad 16: Net-(R6-Pad2) -> /LED_D2
- U1 pad 17: Net-(R7-Pad2) -> /LED_D1
- U1 pad 18: (no net) -> /LED_D0
- U2 pad 10: Net-(U1-Pad1) -> Net-(U2-Pad10)
- U2 pad 17: Net-(U2-Pad17) -> Net-(U1-Pad8)
- U2 pad 18: Net-(U2-Pad18) -> Net-(U1-Pad7)
- U2 pad 2: Net-(U1-Pad8) -> Net-(U2-Pad2)
- U2 pad 21: Net-(U2-Pad21) -> Net-(U1-Pad6)
- U2 pad 22: Net-(U2-Pad22) -> Net-(U1-Pad5)
- U2 pad 23: Net-(U2-Pad23) -> Net-(U1-Pad4)
- U2 pad 24: Net-(U2-Pad24) -> Net-(U1-Pad3)
- U2 pad 25: Net-(U2-Pad25) -> Net-(U1-Pad2)
- U2 pad 26: Net-(U2-Pad26) -> Net-(U1-Pad1)
- U2 pad 3: Net-(U1-Pad7) -> Net-(U2-Pad3)
- U2 pad 4: Net-(U1-Pad6) -> Net-(U2-Pad4)
- U2 pad 5: Net-(U1-Pad5) -> Net-(U2-Pad5)
- U2 pad 6: Net-(U1-Pad4) -> Net-(U2-Pad6)
- U2 pad 7: Net-(U1-Pad3) -> Net-(U2-Pad7)
- U2 pad 9: Net-(U1-Pad2) -> Net-(U2-Pad9)
- U3 pad 1: Net-(U2-Pad26) -> Net-(U2-Pad10)
- U3 pad 11: (no net) -> Net-(R1-Pad2)
- U3 pad 12: /LED_D6 -> Net-(R2-Pad2)
- U3 pad 13: /LED_D5 -> Net-(R3-Pad2)
- U3 pad 14: /LED_D4 -> Net-(R4-Pad2)
- U3 pad 15: /LED_D3 -> Net-(R5-Pad2)
- U3 pad 16: /LED_D2 -> Net-(R6-Pad2)
- U3 pad 17: /LED_D1 -> Net-(R7-Pad2)
- U3 pad 18: /LED_D0 -> (no net)
- U3 pad 2: Net-(U2-Pad25) -> Net-(U2-Pad9)
- U3 pad 3: Net-(U2-Pad24) -> Net-(U2-Pad7)
- U3 pad 4: Net-(U2-Pad23) -> Net-(U2-Pad6)
- U3 pad 5: Net-(U2-Pad22) -> Net-(U2-Pad5)
- U3 pad 6: Net-(U2-Pad21) -> Net-(U2-Pad4)
- U3 pad 7: Net-(U2-Pad18) -> Net-(U2-Pad3)
- U3 pad 8: Net-(U2-Pad17) -> Net-(U2-Pad2)
Routing:
- net VDD: track 126.0 -> 169.1 mm, vias 4 -> 7
- net Net-(U2-Pad18): track 30.0 -> 0.00 mm, vias 2 -> 0
- net Net-(U1-Pad7): track 5.08 -> 33.0 mm, vias 0 -> 2
- net Net-(U2-Pad17): track 16.3 -> 0.00 mm
- net Net-(U1-Pad8): track 5.08 -> 16.3 mm, vias 0 -> 2
- net Net-(U2-Pad10): track 0.00 -> 7.62 mm
- net Net-(U2-Pad9): track 0.00 -> 7.62 mm
- net Net-(U2-Pad26): track 7.62 -> 0.00 mm
- net Net-(U2-Pad25): track 7.62 -> 0.00 mm
- net Net-(U2-Pad24): track 7.62 -> 0.00 mm
- net Net-(U2-Pad23): track 7.62 -> 0.00 mm
- net Net-(U2-Pad22): track 7.62 -> 0.00 mm
- net Net-(U2-Pad21): track 7.62 -> 0.00 mm
- net GND: track 150.9 -> 156.4 mm, vias 3 -> 6
- net Net-(U2-Pad7): track 0.00 -> 5.08 mm
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
Commit message: メイン飛んだ
Parts:
- removed C1, C2: 0.1u, Capacitor_THT:C_Disc_D3.0mm_W1.6mm_P2.50mm
- removed C3: 0.01u, Capacitor_THT:C_Disc_D3.0mm_W2.0mm_P2.50mm
- removed C4: 10u, Capacitor_THT:CP_Radial_D5.0mm_P2.50mm
- removed R10, R9: 4.7k, Resistor_THT:R_Axial_DIN0204_L3.6mm_D1.6mm_P7.62mm_Horizontal
- removed R8: 10k, Resistor_THT:R_Axial_DIN0204_L3.6mm_D1.6mm_P7.62mm_Horizontal
- removed U1: TBD62783A, Package_DIP:DIP-18_W7.62mm
- removed U2: PIC16F18854-SO, Package_DIP:DIP-28_W7.62mm
- removed U3: ULN2803A, Package_DIP:DIP-18_W7.62mm
- J1: value Conn_PIC_ICSP_ICD -> Conn_01x07_Male; footprint Connector_PinHeader_2.54mm:PinHeader_1x06_P2.54mm_Horizontal -> Connector_PinHeader_2.54mm:PinHeader_1x07_P2.54mm_Vertical
- J2: value Conn_01x04_Male -> Conn_01x07_Male; footprint Connector_PinHeader_2.54mm:PinHeader_1x04_P2.54mm_Horizontal -> Connector_PinHeader_2.54mm:PinHeader_1x07_P2.54mm_Vertical
- moved J1 81.4 mm to (71.1, 101.6), turned to 180 degrees
- moved D1 67.5 mm to (73.7, 106.7), turned to 0 degrees
- moved D2 67.5 mm to (127.0, 106.7), turned to 0 degrees
- moved D3 67.5 mm to (109.2, 106.7), turned to 0 degrees
- moved D4 67.5 mm to (91.4, 106.7), turned to 0 degrees
- moved J2 52.4 mm to (114.3, 88.9), turned to 0 degrees
- moved AFF1 37.5 mm to (78.7, 81.3)
- moved AFF2 37.5 mm to (91.4, 81.3)
- moved AFF3 37.5 mm to (104.1, 81.3)
- moved AFF4 29.6 mm to (86.4, 101.6)
- moved AFF5 29.6 mm to (99.1, 101.6)
- moved R1 25.0 mm to (83.8, 86.4), turned to 180 degrees
- moved R2 22.7 mm to (83.8, 88.9), turned to 180 degrees
- moved BAR1 21.6 mm to (127.0, 94.0)
- moved R3 20.5 mm to (83.8, 91.4), turned to 180 degrees
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Connections:
- J1 pad 2: VDD -> Net-(J1-Pad2)
- J1 pad 3: GND -> Net-(J1-Pad3)
- J1 pad 6: (no net) -> Net-(J1-Pad6)
- J2 pad 1: VDD -> /LED_D0
- J2 pad 2: /SDA -> /LED_D1
- J2 pad 3: /SCL -> /LED_D2
- J2 pad 4: GND -> /LED_D3
- R1 pad 2: Net-(R1-Pad2) -> Net-(J1-Pad7)
- R2 pad 2: Net-(R2-Pad2) -> Net-(J1-Pad6)
- R3 pad 2: Net-(R3-Pad2) -> Net-(J1-Pad5)
- R4 pad 2: Net-(R4-Pad2) -> Net-(J1-Pad4)
- R5 pad 2: Net-(R5-Pad2) -> Net-(J1-Pad3)
- R6 pad 2: Net-(R6-Pad2) -> Net-(J1-Pad2)
- R7 pad 2: Net-(R7-Pad2) -> Net-(J1-Pad1)
Routing:
- net VDD: track 169.1 -> 0.00 mm, vias 7 -> 0
- net GND: track 156.4 -> 0.00 mm, vias 6 -> 0
- net /LED_D6: track 152.4 -> 81.9 mm, vias 1 -> 4
- net /LED_S1: track 186.7 -> 119.0 mm, vias 9 -> 7
- net /LED_D4: track 86.9 -> 30.7 mm, vias 0 -> 2
- net /LED_S3: track 172.5 -> 119.5 mm, vias 8 -> 5
- net /LED_S0: track 166.2 -> 115.7 mm
- net /SDA: track 45.7 -> 0.00 mm, vias 2 -> 0
- net /LED_S4: track 175.0 -> 133.7 mm, vias 9 -> 1
- net /LED_S5: track 179.3 -> 142.3 mm, vias 8 -> 6
- net /SCL: track 35.6 -> 0.00 mm
- net /LED_D1: track 51.5 -> 16.3 mm
- net /LED_D2: track 51.7 -> 16.7 mm, vias 0 -> 1
- net Net-(U1-Pad7): track 33.0 -> 0.00 mm, vias 2 -> 0
- net /LED_D3: track 62.8 -> 30.8 mm
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Other:
- board outline added: 71.1 x 45.7 mm
- board text removed: "25x40"
