File: Circuit/Display/Display.sch (KiCad schematic (older format))
At the start: 29 parts, among them J1 Conn_PIC_ICSP_ICD, J2 Conn_01x04_Female, U1 TBD62783A, U2 PIC16F18854-SO, U3 ULN2803A

Commit message: display
Connections:
- net LED_D0: no longer AFF1.8 (C.A.)
- net LED_D1: no longer AFF3.8 (C.A.)
- net LED_D2: no longer AFF5.3 (C.A.)
- net LED_D3: no longer AFF2.8 (C.A.)
- net LED_D4: no longer AFF4.3 (C.A.)
- no-connect marks 9 -> 13
Changed lines of the file:
@@
 Text Label 6300 5300 2    50   ~ 0
 LED_D1
-Text Label 8200 5300 2    50   ~ 0
+Text Label 8200 5200 2    50   ~ 0
 LED_D2
 Text Label 4400 6550 2    50   ~ 0
 LED_D3
-Text Label 6300 6550 2    50   ~ 0
+Text Label 6300 6450 2    50   ~ 0
 LED_D4
 Text Label 2500 5650 2    50   ~ 0
@@
 	2800 5800 3100 5800
 Wire Wire Line
-	4100 5200 4100 5300
-Wire Wire Line
 	4100 5300 4400 5300
-Connection ~ 4100 5300
 Entry Wire Line
 	2700 6350 2800 6450
@@
 	2800 7050 3100 7050
 Wire Wire Line
-	4100 6450 4100 6550
-Wire Wire Line
 	4100 6550 4400 6550
-Connection ~ 4100 6550
 NoConn ~ 4100 5900
 NoConn ~ 4100 7150
@@
 	4700 5800 5000 5800
 Wire Wire Line
-	6000 5200 6000 5300
-Wire Wire Line
 	6000 5300 6300 5300
-Connection ~ 6000 5300
 Entry Wire Line
 	4600 6350 4700 6450
@@
 LED_S6
 Entry Wire Line
-	6300 6550 6400 6650
-$Comp
-L Display_Character:LTS-6960HR AFF4
-U 1 1 60B00F71
-P 5500 6850
-F 0 "AFF4" H 5500 7517 50  0000 C CNN
-F 1 "LTS-6960HR" H 5500 7426 50  0000 C CNN
-F 2 "Display_7Segment:7SegmentLED_LTS6760_LTS6780" H 5500 6250 50  0001 C CNN
-F 3 "https://datasheet.octopart.com/LTS-6960HR-Lite-On-datasheet-11803242.pdf" H 5500 6850 50  0001 C CNN
-	1    5500 6850
-	1    0    0    -1
-$EndComp
+	6300 6450 6400 6550
 Wire Wire Line
 	4700 6450 5000 6450
@@
 Wire Wire Line
 	4700 7050 5000 7050
-Wire Wire Line
-	6000 6450 6000 6550
-Wire Wire Line
-	6000 6550 6300 6550
-Connection ~ 6000 6550
 NoConn ~ 6000 5900
 NoConn ~ 6000 7150
@@
 LED_S6
 Entry Wire Line
-	8200 5300 8300 5400
+	8200 5200 8300 5300
 $Comp
 L Display_Character:LTS-6960HR AFF5
@@
 Wire Wire Line
 	6600 5800 6900 5800
-Wire Wire Line
-	7900 5200 7900 5300
-Wire Wire Line
-	7900 5300 8200 5300
-Connection ~ 7900 5300
 NoConn ~ 7900 5900
 Wire Bus Line
 	6500 4700 4600 4700
 Connection ~ 4600 4700
-Wire Bus Line
-	8300 5400 8300 4500
 Connection ~ 8300 4500
 Wire Bus Line
@@
 Wire Wire Line
 	3550 3450 3750 3450
-Wire Bus Line
-	2600 4500 2600 7350
-Wire Bus Line
-	4500 4500 4500 6650
-Wire Bus Line
-	6400 4500 6400 6650
-Wire Bus Line
-	1200 2350 1200 4700
-Wire Bus Line
-	8850 2750 8850 4500
-Wire Bus Line
-	6500 4700 6500 5700
-Wire Bus Line
-	1200 4700 1200 7150
-Wire Bus Line
-	2700 4700 2700 6950
-Wire Bus Line
-	4600 4700 4600 6950
-$Comp
-L power:GND #PWR?
+$Comp
+L power:GND #PWR0101
 U 1 1 60CC475E
 P 3550 3450
-F 0 "#PWR?" H 3550 3200 50  0001 C CNN
+F 0 "#PWR0101" H 3550 3200 50  0001 C CNN
 F 1 "GND" H 3555 3277 50  0000 C CNN
 F 2 "" H 3550 3450 50  0001 C CNN
@@
 $EndComp
 $Comp
-L power:GND #PWR?
+L power:GND #PWR0102
 U 1 1 60CC507C
 P 4850 3650
-F 0 "#PWR?" H 4850 3400 50  0001 C CNN
+F 0 "#PWR0102" H 4850 3400 50  0001 C CNN
 F 1 "GND" H 4855 3477 50  0000 C CNN
 F 2 "" H 4850 3650 50  0001 C CNN
@@
 	1    0    0    -1
 $EndComp
+NoConn ~ 6000 5200
+NoConn ~ 4100 6450
+$Comp
+L Display_Character:LTS-6960HR AFF4
+U 1 1 60B00F71
+P 5500 6850
+F 0 "AFF4" H 5500 7517 50  0000 C CNN
+F 1 "LTS-6960HR" H 5500 7426 50  0000 C CNN
+F 2 "Display_7Segment:7SegmentLED_LTS6760_LTS6780" H 5500 6250 50  0001 C CNN
+F 3 "https://datasheet.octopart.com/LTS-6960HR-Lite-On-datasheet-11803242.pdf" H 5500 6850 50  0001 C CNN
+	1    5500 6850
+	1    0    0    -1
+$EndComp
+NoConn ~ 6000 6550
+NoConn ~ 7900 5300
+Wire Wire Line
+	6000 6450 6300 6450
+Wire Wire Line
+	8200 5200 7900 5200
+Wire Bus Line
+	8300 4500 8300 5400
+Wire Bus Line
+	2600 4500 2600 7350
+Wire Bus Line
+	4500 4500 4500 6650
+Wire Bus Line
+	6400 4500 6400 6650
+Wire Bus Line
+	1200 2350 1200 4700
+Wire Bus Line
+	8850 2750 8850 4500
+Wire Bus Line
+	6500 4700 6500 5700
+Wire Bus Line
+	1200 4700 1200 7150
+Wire Bus Line
+	2700 4700 2700 6950
+Wire Bus Line
+	4600 4700 4600 6950
 $EndSCHEMATC

Commit message: 20200223
Parts:
- R1: value 4.7k -> 220
Other:
- moved on the sheet: AFF1, AFF2, AFF3, AFF4, AFF5, BAR1, C1, C2, C3, C4, D1, D2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

Commit message: mother回路図作成
Parts:
- C4: symbol Device:C -> Device:CP
- J1: footprint Connector_PinHeader_2.54mm:PinHeader_1x06_P2.54mm_Vertical -> Connector_PinHeader_2.54mm:PinHeader_1x06_P2.54mm_Horizontal
- J2: footprint Connector_PinSocket_2.54mm:PinSocket_1x04_P2.54mm_Vertical -> Connector_PinHeader_2.54mm:PinHeader_1x04_P2.54mm_Horizontal; symbol Connector:Conn_01x04_Female -> Connector:Conn_01x04_Male
- R2, R3, R4, R5, R6, R7: value 4.7k -> 220
Connections:
- net GND: now also C4.2; no longer C4.1
- net VDD: now also C4.1; no longer C4.2
- net SCL: now reaches J2.3 (Pin_3), R9.2, U2.14 (RC3)
- net SDA: now reaches J2.2 (Pin_2), R10.2, U2.15 (RC4)
Changed lines of the file:
@@
 	1    0    0    -1
 $EndComp
-Wire Wire Line
-	7750 6450 7850 6450
-Connection ~ 7850 6450
-$Comp
-L Device:C C4
+$Comp
+L Device:CP C4
 U 1 1 608EC962
 P 7850 6600
@@
 F 3 "~" H 7850 6600 50  0001 C CNN
 	1    7850 6600
-	-1   0    0    1
+	1    0    0    -1
 $EndComp
 Wire Wire Line
@@
 	1    0    0    -1
 $EndComp
-Wire Wire Line
-	9050 6750 9350 6750
 $Comp
 L power:PWR_FLAG #FLG02
@@
 	-1   0    0    1
 $EndComp
-Wire Wire Line
-	7850 6450 9050 6450
-Wire Wire Line
-	9050 6450 9350 6450
 Connection ~ 9050 6450
 $Comp
@@
 Wire Wire Line
 	8500 6750 9050 6750
-Wire Wire Line
-	8300 6650 9350 6650
-Wire Wire Line
-	8200 6550 9350 6550
 $Comp
 L power:GND #PWR014
@@
 Wire Wire Line
 	8200 6550 8200 7000
-$Comp
-L Connector:Conn_01x04_Female J2
-U 1 1 607881ED
-P 9550 6550
-F 0 "J2" H 9578 6526 50  0000 L CNN
-F 1 "Conn_01x04_Female" H 9578 6435 50  0000 L CNN
-F 2 "Connector_PinSocket_2.54mm:PinSocket_1x04_P2.54mm_Vertical" H 9550 6550 50  0001 C CNN
-F 3 "~" H 9550 6550 50  0001 C CNN
-	1    9550 6550
-	1    0    0    -1
-$EndComp
 $Comp
 L Device:R R1
@@
 F 0 "J1" H 7020 4396 50  0000 R CNN
 F 1 "Conn_PIC_ICSP_ICD" H 7020 4305 50  0000 R CNN
-F 2 "Connector_PinHeader_2.54mm:PinHeader_1x06_P2.54mm_Vertical" H 7400 4500 50  0001 C CNN
+F 2 "Connector_PinHeader_2.54mm:PinHeader_1x06_P2.54mm_Horizontal" H 7400 4500 50  0001 C CNN
 F 3 "http://ww1.microchip.com/downloads/en/devicedoc/30277d.pdf" V 7050 4200 50  0001 C CNN
 	1    7350 4350
@@
 P 3250 5800
 F 0 "R7" V 3300 5600 50  0000 C CNN
-F 1 "4.7k" V 3300 5400 50  0000 C CNN
+F 1 "220" V 3300 5400 50  0000 C CNN
 F 2 "Resistor_THT:R_Axial_DIN0204_L3.6mm_D1.6mm_P7.62mm_Horizontal" V 3180 5800 50  0001 C CNN
 F 3 "~" H 3250 5800 50  0001 C CNN
@@
 P 3250 5700
 F 0 "R6" V 3300 5500 50  0000 C CNN
-F 1 "4.7k" V 3300 5300 50  0000 C CNN
+F 1 "220" V 3300 5300 50  0000 C CNN
 F 2 "Resistor_THT:R_Axial_DIN0204_L3.6mm_D1.6mm_P7.62mm_Horizontal" V 3180 5700 50  0001 C CNN
 F 3 "~" H 3250 5700 50  0001 C CNN
@@
 P 3250 5600
 F 0 "R5" V 3300 5400 50  0000 C CNN
-F 1 "4.7k" V 3300 5200 50  0000 C CNN
+F 1 "220" V 3300 5200 50  0000 C CNN
 F 2 "Resistor_THT:R_Axial_DIN0204_L3.6mm_D1.6mm_P7.62mm_Horizontal" V 3180 5600 50  0001 C CNN
 F 3 "~" H 3250 5600 50  0001 C CNN
@@
 P 3250 5500
 F 0 "R4" V 3300 5300 50  0000 C CNN
-F 1 "4.7k" V 3300 5100 50  0000 C CNN
+F 1 "220" V 3300 5100 50  0000 C CNN
 F 2 "Resistor_THT:R_Axial_DIN0204_L3.6mm_D1.6mm_P7.62mm_Horizontal" V 3180 5500 50  0001 C CNN
 F 3 "~" H 3250 5500 50  0001 C CNN
@@
 P 3250 5400
 F 0 "R3" V 3300 5200 50  0000 C CNN
-F 1 "4.7k" V 3300 5000 50  0000 C CNN
+F 1 "220" V 3300 5000 50  0000 C CNN
 F 2 "Resistor_THT:R_Axial_DIN0204_L3.6mm_D1.6mm_P7.62mm_Horizontal" V 3180 5400 50  0001 C CNN
 F 3 "~" H 3250 5400 50  0001 C CNN
@@
 P 3250 5300
 F 0 "R2" V 3300 5100 50  0000 C CNN
-F 1 "4.7k" V 3300 4900 50  0000 C CNN
+F 1 "220" V 3300 4900 50  0000 C CNN
 F 2 "Resistor_THT:R_Axial_DIN0204_L3.6mm_D1.6mm_P7.62mm_Horizontal" V 3180 5300 50  0001 C CNN
 F 3 "~" H 3250 5300 50  0001 C CNN
@@
 	0    -1   -1   0
 $EndComp
+Wire Wire Line
+	7750 6450 7850 6450
+Connection ~ 7850 6450
+Wire Wire Line
+	7850 6450 9050 6450
+Wire Wire Line
+	9800 6450 9800 6350
+Wire Wire Line
+	9050 6450 9800 6450
+Wire Wire Line
+	9700 6350 9700 6550
+Wire Wire Line
+	8200 6550 9700 6550
+Wire Wire Line
+	9600 6650 9600 6350
+Wire Wire Line
+	8300 6650 9600 6650
+Wire Wire Line
+	9500 6350 9500 6750
+Wire Wire Line
+	9050 6750 9500 6750
+$Comp
+L Connector:Conn_01x04_Male J2
+U 1 1 607881ED
+P 9700 6150
+F 0 "J2" H 9728 6126 50  0000 L CNN
+F 1 "Conn_01x04_Female" H 9728 6035 50  0000 L CNN
+F 2 "Connector_PinHeader_2.54mm:PinHeader_1x04_P2.54mm_Horizontal" H 9700 6150 50  0001 C CNN
+F 3 "~" H 9700 6150 50  0001 C CNN
+	1    9700 6150
+	0    1    1    0
+$EndComp
 Wire Bus Line
 	4100 7250 4100 10100
@@
 Wire Bus Line
 	4200 7450 4200 9700
+Text Label 9200 6550 0    50   ~ 0
+SDA
+Text Label 9200 6650 0    50   ~ 0
+SCL
 $EndSCHEMATC

Commit message: 回路完成
Parts:
- J2: value Conn_01x04_Female -> Conn_01x04_Male
Connections:
- net LED_D0: now also U1.18 (O1); no longer U3.18 (O1)
- net LED_D1: now also U1.17 (O2); no longer U3.17 (O2)
- net LED_D2: now also U1.16 (O3); no longer U3.16 (O3)
- net LED_D3: now also U1.15 (O4); no longer U3.15 (O4)
- net LED_D4: now also U1.14 (O5); no longer U3.14 (O5)
- net LED_D5: now also BAR1.10 (A), BAR1.4 (A), BAR1.5 (A), BAR1.6 (A), BAR1.7 (A), BAR1.8 (A), BAR1.9 (A), U1.13 (O6); no longer BAR1.14 (K), BAR1.15 (K), BAR1.16 (K), BAR1.17 (K), BAR1.18 (K), BAR1.19 (K), BAR1.20 (K), U3.13 (O6)
- net LED_D6: now also BAR1.1 (A), BAR1.2 (A), BAR1.3 (A), D1.2 (A), D2.2 (A), D3.2 (A), D4.2 (A), U1.12 (O7); no longer BAR1.11 (K), BAR1.12 (K), BAR1.13 (K), D1.1 (K), D2.1 (K), D3.1 (K), D4.1 (K), U3.12 (O7)
- net LED_S0: now also BAR1.11 (K), BAR1.18 (K); no longer BAR1.1 (A), BAR1.8 (A)
- net LED_S1: now also BAR1.12 (K), BAR1.19 (K); no longer BAR1.2 (A), BAR1.9 (A)
- net LED_S2: now also BAR1.13 (K), BAR1.20 (K); no longer BAR1.10 (A), BAR1.3 (A)
- net LED_S3: now also BAR1.14 (K), D1.1 (K); no longer BAR1.4 (A), D1.2 (A)
- net LED_S4: now also BAR1.15 (K), D2.1 (K); no longer BAR1.5 (A), D2.2 (A)
- net LED_S5: now also BAR1.16 (K), D3.1 (K); no longer BAR1.6 (A), D3.2 (A)
- net LED_S6: now also BAR1.17 (K), D4.1 (K); no longer BAR1.7 (A), D4.2 (A)
- net at U2.10 (RA6): now also U3.1 (I1); no longer U1.1 (I1)
- net at U2.17 (RC6): now also U1.8 (I8); no longer U3.8 (I8)
- net at U2.18 (RC7): now also U1.7 (I7); no longer U3.7 (I7)
- net at U2.2 (RA0): now also U3.8 (I8); no longer U1.8 (I8)
- net at U2.21 (RB0): now also U1.6 (I6); no longer U3.6 (I6)
- net at U2.22 (RB1): now also U1.5 (I5); no longer U3.5 (I5)
- net at U2.23 (RB2): now also U1.4 (I4); no longer U3.4 (I4)
- net at U2.24 (RB3): now also U1.3 (I3); no longer U3.3 (I3)
- net at U2.25 (RB4): now also U1.2 (I2); no longer U3.2 (I2)
- net at U2.26 (RB5): now also U1.1 (I1); no longer U3.1 (I1)
- net at U2.3 (RA1): now also U3.7 (I7); no longer U1.7 (I7)
- net at U2.4 (RA2): now also U3.6 (I6); no longer U1.6 (I6)
- net at U2.5 (RA3): now also U3.5 (I5); no longer U1.5 (I5)
- net at U2.6 (RA4): now also U3.4 (I4); no longer U1.4 (I4)
- net at U2.7 (RA5): now also U3.3 (I3); no longer U1.3 (I3)
- net at U2.9 (RA7): now also U3.2 (I2); no longer U1.2 (I2)
- net at U1.11 (O8): no longer R1.2
- net at R2.2: now also U3.12 (O7); no longer U1.12 (O7)
- net at R3.2: now also U3.13 (O6); no longer U1.13 (O6)
- net at R4.2: now also U3.14 (O5); no longer U1.14 (O5)
- net at R5.2: now also U3.15 (O4); no longer U1.15 (O4)
- net at R6.2: now also U3.16 (O3); no longer U1.16 (O3)
- net at R7.2: now also U3.17 (O2); no longer U1.17 (O2)
- net at U3.11 (O8): now also R1.2
Other:
- moved on the sheet: C1, D1, D2, D3, D4, U1, U3
Changed lines of the file:
@@
 	4700 5900 5100 5900
 Wire Wire Line
-	4300 4500 3800 4500
-Wire Wire Line
-	4300 5000 4300 4500
-Wire Wire Line
-	4300 6500 4300 6100
-Wire Wire Line
-	3800 6500 4300 6500
+	7350 4800 7350 5050
 $Comp
 L Device:LED D4
@@
 F 3 "~" H 3450 10000 50  0001 C CNN
 	1    3450 10000
-	-1   0    0    1
+	1    0    0    -1
 $EndComp
 $Comp
@@
 F 3 "~" H 3450 9700 50  0001 C CNN
 	1    3450 9700
-	-1   0    0    1
+	1    0    0    -1
 $EndComp
 $Comp
@@
 F 3 "~" H 3450 9400 50  0001 C CNN
 	1    3450 9400
-	-1   0    0    1
+	1    0    0    -1
 $EndComp
 Wire Bus Line
@@
 	4300 7950 4600 7950
 Wire Wire Line
-	3700 8400 4000 8400
-Wire Wire Line
 	4000 10000 3700 10000
 $Comp
@@
 	-1   0    0    1
 $EndComp
-Wire Wire Line
-	3800 6250 3800 6500
 $Comp
 L power:GND #PWR01
 U 1 1 60812496
-P 3500 6500
-F 0 "#PWR01" H 3500 6250 50  0001 C CNN
-F 1 "GND" H 3505 6327 50  0000 C CNN
-F 2 "" H 3500 6500 50  0001 C CNN
-F 3 "" H 3500 6500 50  0001 C CNN
-	1    3500 6500
-	1    0    0    -1
-$EndComp
-Connection ~ 3800 6500
+P 7650 5050
+F 0 "#PWR01" H 7650 4800 50  0001 C CNN
+F 1 "GND" H 7655 4877 50  0000 C CNN
+F 2 "" H 7650 5050 50  0001 C CNN
+F 3 "" H 7650 5050 50  0001 C CNN
+	1    7650 5050
+	1    0    0    -1
+$EndComp
 $Comp
 L Device:C C1
 U 1 1 60811A21
-P 3650 6500
-F 0 "C1" V 3398 6500 50  0000 C CNN
-F 1 "0.1u" V 3489 6500 50  0000 C CNN
-F 2 "Capacitor_THT:C_Disc_D3.0mm_W1.6mm_P2.50mm" H 3688 6350 50  0001 C CNN
-F 3 "~" H 3650 6500 50  0001 C CNN
-	1    3650 6500
-	0    1    1    0
+P 7500 5050
+F 0 "C1" V 7248 5050 50  0000 C CNN
+F 1 "0.1u" V 7339 5050 50  0000 C CNN
+F 2 "Capacitor_THT:C_Disc_D3.0mm_W1.6mm_P2.50mm" H 7538 4900 50  0001 C CNN
+F 3 "~" H 7500 5050 50  0001 C CNN
+	1    7500 5050
+	0    -1   -1   0
 $EndComp
 Connection ~ 5750 4500
@@
 L power:VDD #PWR02
 U 1 1 607FC6E4
-P 3800 6250
-F 0 "#PWR02" H 3800 6100 50  0001 C CNN
-F 1 "VDD" H 3815 6423 50  0000 C CNN
-F 2 "" H 3800 6250 50  0001 C CNN
-F 3 "" H 3800 6250 50  0001 C CNN
-	1    3800 6250
+P 7350 4800
+F 0 "#PWR02" H 7350 4650 50  0001 C CNN
+F 1 "VDD" H 7365 4973 50  0000 C CNN
+F 2 "" H 7350 4800 50  0001 C CNN
+F 3 "" H 7350 4800 50  0001 C CNN
+	1    7350 4800
 	1    0    0    -1
 $EndComp
@@
 	1    0    0    -1
 $EndComp
-NoConn ~ 7750 5300
 NoConn ~ 7750 6100
 NoConn ~ 3900 5900
@@
 Wire Wire Line
 	3700 9100 3700 9400
-Connection ~ 3700 9100
 Wire Wire Line
 	3600 9100 3700 9100
@@
 LED_S0
 Wire Wire Line
-	3300 8400 2800 8400
-Wire Wire Line
 	2800 8300 3300 8300
 Wire Wire Line
@@
 Wire Wire Line
 	2800 8100 3300 8100
-Wire Wire Line
-	3300 8000 2800 8000
 Wire Wire Line
 	2800 7900 3300 7900
@@
 L Transistor_Array:ULN2803A U3
 U 1 1 6035D1F1
-P 7350 5600
-F 0 "U3" H 7350 6167 50  0000 C CNN
-F 1 "ULN2803A" H 7350 6076 50  0000 C CNN
-F 2 "Package_DIP:DIP-18_W7.62mm" H 7400 4950 50  0001 L CNN
-F 3 "http://www.ti.com/lit/ds/symlink/uln2803a.pdf" H 7450 5400 50  0001 C CNN
-	1    7350 5600
-	1    0    0    -1
+P 4300 5700
+F 0 "U3" H 4300 6267 50  0000 C CNN
+F 1 "ULN2803A" H 4300 6176 50  0000 C CNN
+F 2 "Package_DIP:DIP-18_W7.62mm" H 4350 5050 50  0001 L CNN
+F 3 "http://www.ti.com/lit/ds/symlink/uln2803a.pdf" H 4400 5500 50  0001 C CNN
+	1    4300 5700
+	-1   0    0    1
 $EndComp
 $Comp
 L Transistor_Array:TBD62783A U1
 U 1 1 60340DE8
-P 4300 5600
-F 0 "U1" H 4300 4819 50  0000 C CNN
-F 1 "TBD62783A" H 4300 4910 50  0000 C CNN
-F 2 "Package_DIP:DIP-18_W7.62mm" H 4300 5050 50  0001 C CNN
-F 3 "http://toshiba.semicon-storage.com/info/docget.jsp?did=30523&prodName=TBD62783APG" H 4000 6000 50  0001 C CNN
-	1    4300 5600
-	-1   0    0    1
-$EndComp
-Wire Wire Line
-	3700 7800 3700 7900
-Connection ~ 3700 7900
-Wire Wire Line
-	3700 7900 3700 8000
-Connection ~ 3700 8000
-Wire Wire Line
-	3700 8000 3700 8100
-Connection ~ 3700 8100
-Wire Wire Line
-	3700 8100 3700 8200
-Connection ~ 3700 8200
-Wire Wire Line
-	3700 8300 3700 8400
-Wire Wire Line
-	3700 8200 3700 8300
-Connection ~ 3700 8300
-Connection ~ 3700 8400
-Wire Wire Line
-	3700 8500 3700 8600
-Connection ~ 3700 8600
-Wire Wire Line
-	3700 9100 3700 8700
-Wire Wire Line
-	3700 8600 3700 8700
-Connection ~ 3700 8700
-$Comp
-L LED:HDSP-4830_2 BAR1
-U 1 1 60332800
-P 3500 8200
-F 0 "BAR1" H 3500 8867 50  0000 C CNN
-F 1 "HDSP-4830_2" H 3500 8776 50  0000 C CNN
-F 2 "Display:HDSP-4830" H 3500 7400 50  0001 C CNN
-F 3 "https://docs.broadcom.com/docs/AV02-1798EN" H 1500 8400 50  0001 C CNN
-	1    3500 8200
+P 7350 5700
+F 0 "U1" H 7350 4919 50  0000 C CNN
+F 1 "TBD62783A" H 7350 5010 50  0000 C CNN
+F 2 "Package_DIP:DIP-18_W7.62mm" H 7350 5150 50  0001 C CNN
+F 3 "http://toshiba.semicon-storage.com/info/docget.jsp?did=30523&prodName=TBD62783APG" H 7050 6100 50  0001 C CNN
+	1    7350 5700
 	1    0    0    -1
 $EndComp
@@
 F 3 "~" H 3450 9100 50  0001 C CNN
 	1    3450 9100
-	-1   0    0    1
+	1    0    0    -1
 $EndComp
 Wire Wire Line
@@
 $EndComp
 Wire Wire Line
-	7350 6300 7350 6500
+	4300 5000 4300 4800
 $Comp
 L power:GND #PWR09
 U 1 1 602E59D5
-P 7350 6500
-F 0 "#PWR09" H 7350 6250 50  0001 C CNN
-F 1 "GND" H 7355 6327 50  0000 C CNN
-F 2 "" H 7350 6500 50  0001 C CNN
-F 3 "" H 7350 6500 50  0001 C CNN
-	1    7350 6500
+P 4000 4800
+F 0 "#PWR09" H 4000 4550 50  0001 C CNN
+F 1 "GND" H 4005 4627 50  0000 C CNN
+F 2 "" H 4000 4800 50  0001 C CNN
+F 3 "" H 4000 4800 50  0001 C CNN
+	1    4000 4800
 	1    0    0    -1
 $EndComp
@@
 	1    0    0    -1
 $EndComp
-Wire Wire Line
-	3800 4500 3800 4700
 $Comp
 L power:GND #PWR03
 U 1 1 602E0BCF
-P 3800 4700
-F 0 "#PWR03" H 3800 4450 50  0001 C CNN
-F 1 "GND" H 3805 4527 50  0000 C CNN
-F 2 "" H 3800 4700 50  0001 C CNN
-F 3 "" H 3800 4700 50  0001 C CNN
-	1    3800 4700
+P 7350 6300
+F 0 "#PWR03" H 7350 6050 50  0001 C CNN
+F 1 "GND" H 7355 6127 50  0000 C CNN
+F 2 "" H 7350 6300 50  0001 C CNN
+F 3 "" H 7350 6300 50  0001 C CNN
+	1    7350 6300
 	1    0    0    -1
 $EndComp
@@
 P 9700 6150
 F 0 "J2" H 9728 6126 50  0000 L CNN
-F 1 "Conn_01x04_Female" H 9728 6035 50  0000 L CNN
+F 1 "Conn_01x04_Male" H 9728 6035 50  0000 L CNN
 F 2 "Connector_PinHeader_2.54mm:PinHeader_1x04_P2.54mm_Horizontal" H 9700 6150 50  0001 C CNN
 F 3 "~" H 9700 6150 50  0001 C CNN
@@
 	0    1    1    0
 $EndComp
-Wire Bus Line
-	4100 7250 4100 10100
-Wire Bus Line
-	6000 7250 6000 9400
-Wire Bus Line
-	9800 7250 9800 8150
-Wire Bus Line
-	7900 7250 7900 9400
-Wire Bus Line
-	8000 7450 8000 8450
-Wire Bus Line
-	10350 5500 10350 7250
-Wire Bus Line
-	2700 5100 2700 7450
-Wire Bus Line
-	6100 7450 6100 9700
-Wire Bus Line
-	2700 7450 2700 9900
-Wire Bus Line
-	4200 7450 4200 9700
 Text Label 9200 6550 0    50   ~ 0
 SDA
 Text Label 9200 6650 0    50   ~ 0
 SCL
+Connection ~ 3700 8000
+Connection ~ 3700 9100
+Connection ~ 3700 8700
+Wire Wire Line
+	3700 9100 3700 8700
+Connection ~ 3700 8600
+Wire Wire Line
+	3700 8600 3700 8700
+Wire Wire Line
+	3700 8500 3700 8600
+Connection ~ 3700 8400
+Connection ~ 3700 8300
+Wire Wire Line
+	3700 8200 3700 8300
+Wire Wire Line
+	3700 8300 3700 8400
+Connection ~ 3700 8200
+Connection ~ 3700 8100
+Wire Wire Line
+	3700 8100 3700 8200
+Wire Wire Line
+	3700 8000 3700 8100
+Connection ~ 3700 7900
+Wire Wire Line
+	3700 7900 3700 8000
+Wire Wire Line
+	3700 7800 3700 7900
+Wire Wire Line
+	3700 8400 4000 8400
+Wire Wire Line
+	3300 8400 2800 8400
+Wire Wire Line
+	3300 8000 2800 8000
+$Comp
+L LED:HDSP-4830_2 BAR1
+U 1 1 60332800
+P 3500 8300
+F 0 "BAR1" H 3500 8967 50  0000 C CNN
+F 1 "HDSP-4830_2" H 3500 8876 50  0000 C CNN
+F 2 "Display:HDSP-4830" H 3500 7500 50  0001 C CNN
+F 3 "https://docs.broadcom.com/docs/AV02-1798EN" H 1500 8500 50  0001 C CNN
+	1    3500 8300
+	-1   0    0    1
+$EndComp
+NoConn ~ 3900 6000
+Wire Wire Line
+	4000 4800 4300 4800
+Wire Bus Line
+	4100 7250 4100 10100
+Wire Bus Line
+	6000 7250 6000 9400
+Wire Bus Line
+	9800 7250 9800 8150
+Wire Bus Line
+	7900 7250 7900 9400
+Wire Bus Line
+	8000 7450 8000 8450
+Wire Bus Line
+	10350 5500 10350 7250
+Wire Bus Line
+	2700 5100 2700 7450
+Wire Bus Line
+	6100 7450 6100 9700
+Wire Bus Line
+	2700 7450 2700 9900
+Wire Bus Line
+	4200 7450 4200 9700
+Connection ~ 7350 5050
+Wire Wire Line
+	7350 5050 7350 5200
 $EndSCHEMATC

Commit message: メイン飛んだ
Parts:
- removed C1, C2: 0.1u, Capacitor_THT:C_Disc_D3.0mm_W1.6mm_P2.50mm, symbol Device:C
- removed C3: 0.01u, Capacitor_THT:C_Disc_D3.0mm_W2.0mm_P2.50mm, symbol Device:C
- removed C4: 10u, Capacitor_THT:CP_Radial_D5.0mm_P2.50mm, symbol Device:CP
- removed J1: Conn_PIC_ICSP_ICD, Connector_PinHeader_2.54mm:PinHeader_1x06_P2.54mm_Horizontal, symbol Connector:Conn_PIC_ICSP_ICD
- removed J2: Conn_01x04_Male, Connector_PinHeader_2.54mm:PinHeader_1x04_P2.54mm_Horizontal, symbol Connector:Conn_01x04_Male
- removed R10, R9: 4.7k, Resistor_THT:R_Axial_DIN0204_L3.6mm_D1.6mm_P7.62mm_Horizontal, symbol Device:R
- removed R8: 10k, Resistor_THT:R_Axial_DIN0204_L3.6mm_D1.6mm_P7.62mm_Horizontal, symbol Device:R
- removed U1: TBD62783A, Package_DIP:DIP-18_W7.62mm, symbol Transistor_Array:TBD62783A
- removed U2: PIC16F18854-SO, Package_DIP:DIP-28_W7.62mm, symbol MCU_Microchip_PIC16:PIC16F18854-SO
- removed U3: ULN2803A, Package_DIP:DIP-18_W7.62mm, symbol Transistor_Array:ULN2803A
- added J1, J2: Conn_01x07_Male, Connector_PinHeader_2.54mm:PinHeader_1x07_P2.54mm_Vertical, symbol Connector:Conn_01x07_Male
Connections:
- net LED_D0: now also J2.1 (Pin_1)
- net LED_D1: now also J2.2 (Pin_2)
- net LED_D2: now also J2.3 (Pin_3)
- net LED_D3: now also J2.4 (Pin_4)
- net LED_D4: now also J2.5 (Pin_5)
- net LED_D5: now also J2.6 (Pin_6)
- net LED_D6: now also J2.7 (Pin_7)
- net at R1.2: now also J1.7 (Pin_7)
- net at R2.2: now also J1.6 (Pin_6)
- net at R3.2: now also J1.5 (Pin_5)
- net at R4.2: now also J1.4 (Pin_4)
- net at R5.2: now also J1.3 (Pin_3)
- net at R6.2: now also J1.2 (Pin_2)
- net at R7.2: now also J1.1 (Pin_1)
- no-connect marks 13 -> 9
