File: Circuit/old/Display/Display.sch (KiCad schematic (older format))
At the start: 19 parts, among them J1 Conn_01x07_Male, J2 Conn_01x07_Male

Commit message: メイン飛んだ
Parts:
- removed J1, J2: Conn_01x07_Male, Connector_PinHeader_2.54mm:PinHeader_1x07_P2.54mm_Vertical, symbol Connector:Conn_01x07_Male
- added C1, C2: 0.1u, Capacitor_THT:C_Disc_D3.0mm_W1.6mm_P2.50mm, symbol Device:C
- added C3: 0.01u, Capacitor_THT:C_Disc_D3.0mm_W2.0mm_P2.50mm, symbol Device:C
- added C4: 10u, Capacitor_THT:CP_Radial_D5.0mm_P2.50mm, symbol Device:CP
- added J1: Conn_PIC_ICSP_ICD, Connector_PinHeader_2.54mm:PinHeader_1x06_P2.54mm_Horizontal, symbol Connector:Conn_PIC_ICSP_ICD
- added J2: Conn_01x04_Male, Connector_PinHeader_2.54mm:PinHeader_1x04_P2.54mm_Horizontal, symbol Connector:Conn_01x04_Male
- added R10, R9: 4.7k, Resistor_THT:R_Axial_DIN0204_L3.6mm_D1.6mm_P7.62mm_Horizontal, symbol Device:R
- added R8: 10k, Resistor_THT:R_Axial_DIN0204_L3.6mm_D1.6mm_P7.62mm_Horizontal, symbol Device:R
- added U1: TBD62783A, Package_DIP:DIP-18_W7.62mm, symbol Transistor_Array:TBD62783A
- added U2: PIC16F18854-SO, Package_DIP:DIP-28_W7.62mm, symbol MCU_Microchip_PIC16:PIC16F18854-SO
- added U3: ULN2803A, Package_DIP:DIP-18_W7.62mm, symbol Transistor_Array:ULN2803A
Connections:
- net labels added: GND, SCL, SDA, VDD
- wire segments 93 -> 170
- no-connect marks 9 -> 13
