File: Circuit/old/Mother/Mother.sch (KiCad schematic (older format))
At the start: 57 parts, among them J1 Conn_01x02_Male, J2 Conn_01x05_Male, J3 Conn_02x09_Odd_Even, J4 Conn_01x04_Male, J5 Conn_02x09_Odd_Even, J6 Conn_PIC_ICSP_ICD, J7 Conn_01x05_Male, U1 74HC00, U2 BP5293-33, U3 BP5293-50, U4 PIC32MX110F016B-I_SP, U5 4051, U6 TLP785

Commit message: メイン飛んだ
Parts:
- renumbered C8 to C10, C9 to C11, C10 to C12, C11 to C14, C12 to C15, C13 to C16, C14 to C17, C15 to C18, C16 to C19, C17 to C20, C18 to C21, C19 to C22, C4 to C6, C5 to C7, C6 to C8, C7 to C9, D1 to D3, R9 to R10, R10 to R11, R11 to R12, R12 to R13, R13 to R14, R14 to R15, R15 to R16, R16 to R17, R17 to R18, R18 to R19, R1 to R2, R19 to R20, R20 to R21, R21 to R22, R22 to R23, R2 to R3, R3 to R4, R4 to R5, R5 to R6, R6 to R7, R7 to R8, R8 to R9
Connections:
- net Sheet60D32BD3/SCL: no longer names the net of J4.3 (Pin_3), U4.17 (TCK/RPB8/SCL1/CTED10/PMD4/RB8)
- net Sheet60D32BD3/SDA: no longer names the net of J4.2 (Pin_2), U4.18 (TDO/RPB9/SDA1/CTED4/PMD3/RB9)
